Commit message: [tiger] add tiger v1 config files

File: robots/tiger/robots/octo/v1_default/robot.urdf.xacro (robot description, xacro)
@@ -2,15 +2,17 @@
 <robot
     xmlns:xacro="http://www.ros.org/wiki/xacro" name="hydrusx" >
-  <xacro:include filename="$(find tiger)/urdf/v1/link.urdf.xacro" />
-  <xacro:property name="battery" value="1"/>
-  <xacro:property name="leg" value="1"/>
-  <xacro:tiger_center_link child1="1" child2="3" child3="5" child4="7" leg="${leg}"/>
-  <xacro:tiger_link self="1" child="2" link_type="general" battery="${battery}" leg="${leg}"/>
-  <xacro:tiger_link self="2" child="2" link_type="end"     battery="${battery}" leg="${leg}"/>
-  <xacro:tiger_link self="3" child="4" link_type="general" battery="${battery}" leg="${leg}"/>
-  <xacro:tiger_link self="4" child="4" link_type="end"     battery="${battery}" leg="${leg}"/>
-  <xacro:tiger_link self="5" child="6" link_type="general" battery="${battery}" leg="${leg}"/>
-  <xacro:tiger_link self="6" child="6" link_type="end"     battery="${battery}" leg="${leg}"/>
-  <xacro:tiger_link self="7" child="8" link_type="general" battery="${battery}" leg="${leg}"/>
-  <xacro:tiger_link self="8" child="8" link_type="end"     battery="${battery}" leg="${leg}"/>
+  <xacro:include filename="$(find tiger)/robots/octo/tiger_v1_base.urdf.xacro" />
+  <xacro:tiger_v1/>
+  #### flight controller ####
+  <!-- TODO -->
+  <xacro:extra_module name = "fc" parent = "center_link" visible = "0">
+    <origin xyz="0 0 0" rpy="0 0 0"/>
+    <inertial>
+      <origin xyz="0 0 0" rpy="0 0 0"/>
+      <mass value="0.001"/>
+      <inertia
+          ixx="0.000004" iyy="0.000004" izz="0.000008"
+          ixy="0.000001" ixz="-0.000001" iyz="-0.000000"/>
+    </inertial>
+  </xacro:extra_module>
 </robot>

File: robots/tiger/urdf/v1/common.xacro (robot description, xacro)
@@ -21,5 +21,6 @@
       <origin xyz="${general_link_length* 0.5} 0 0" rpy="0 ${pi / 2} 0"/>
       <geometry>
-        <cylinder radius="${general_link_radius}" length="${general_link_length}"/>
+        <!--cylinder radius="${general_link_radius}" length="${general_link_length}"/-->
+        <box size="0.1 0.1 ${general_link_length}"/>
       </geometry>
     </collision>
@@ -64,6 +65,6 @@
   <xacro:macro name="friction" params="link">
     <gazebo reference="${link}">
-      <mu1>0.1</mu1>
-      <mu2>0.1</mu2>
+      <mu1>0.5</mu1>
+      <mu2>0.5</mu2>
     </gazebo>
   </xacro:macro>

File: robots/tiger/urdf/v1/link.urdf.xacro (robot description, xacro)
@@ -26,6 +26,7 @@
       <dynamics damping="0.8" friction="0.0"/>
     </joint>
+    <xacro:joint_transmission joint="joint${self}_pitch"/>
     <xacro:if value="${leg == 1}">
-      <xacro:extra_module name="joint_junction_leg${self}" parent="joint_junction_link${self}" visible="1" collision="1" model_url="package://tiger/urdf/v1/mesh/leg/leg.dae">
+      <xacro:extra_module name="joint_junction_leg${self}" parent="joint_junction_link${self}" visible="1" collision="0" model_url="package://tiger/urdf/v1/mesh/leg/leg.dae">
         <origin xyz="0 0 -0.0283" rpy="0 ${pi} 0"/>
         <inertial>
@@ -121,8 +122,4 @@
     <xacro:joint_transmission joint="joint${child3}_yaw"/>
     <xacro:joint_transmission joint="joint${child4}_yaw"/>
-    <xacro:joint_transmission joint="joint_${child4}_pitch"/>
-    <xacro:joint_transmission joint="joint_${child4}_pitch"/>
-    <xacro:joint_transmission joint="joint_${child4}_pitch"/>
-    <xacro:joint_transmission joint="joint_${child4}_pitch"/>
   </xacro:macro>
   #### LINK ####
@@ -193,5 +190,5 @@
       <inertial>
         <origin xyz="0 0 0" rpy="0 0 0"/>
-        <mass value="0.0000001"/>
+        <mass value="0.00001"/>
         <inertia
             ixx="0.000001" iyy="0.000001" izz="0.000001"
@@ -258,5 +255,5 @@
     <xacro:if value="${leg == 1}">
       <xacro:if value="${link_type == 'end'}">
-        <xacro:extra_module name="end_leg${self}" parent="link${self}" visible="1" collision="1"
+        <xacro:extra_module name="end_leg${self}" parent="link${self}" visible="1" collision="0"
                             model_url="package://tiger/urdf/v1/mesh/leg/end_leg.dae">
           <origin xyz="0.4835 0.0 0.0" rpy="0 0 0"/>
@@ -274,5 +271,4 @@
     <xacro:unless value="${self == child}">
       <xacro:joint_transmission joint="joint${child}_yaw"/>
-      <xacro:joint_transmission joint="joint${child}_pitch"/>
     </xacro:unless>
     <xacro:joint_transmission joint="gimbal_roll${self}"/>

Commit message: [tiger] fix urdf and param

File: robots/tiger/robots/octo/v1_default/robot.urdf.xacro (robot description, xacro)
@@ -1,5 +1,5 @@
 <?xml version="1.0"?>
 <robot
-    xmlns:xacro="http://www.ros.org/wiki/xacro" name="hydrusx" >
+    xmlns:xacro="http://www.ros.org/wiki/xacro" name="tiger_v1" >
   <xacro:include filename="$(find tiger)/robots/octo/tiger_v1_base.urdf.xacro" />
   <xacro:tiger_v1/>

File: robots/tiger/urdf/v1/common.xacro (robot description, xacro)
@@ -21,6 +21,5 @@
       <origin xyz="${general_link_length* 0.5} 0 0" rpy="0 ${pi / 2} 0"/>
       <geometry>
-        <!--cylinder radius="${general_link_radius}" length="${general_link_length}"/-->
-        <box size="0.1 0.1 ${general_link_length}"/>
+        <cylinder radius="${general_link_radius}" length="${general_link_length}"/>
       </geometry>
     </collision>
@@ -42,9 +41,9 @@
       </xacro:if>
       <xacro:if value="${collision == 1}">
-        <visual>
+        <collision>
           <geometry>
             <mesh filename="${model_url}"/>
           </geometry>
-        </visual>
+        </collision>
       </xacro:if>
     </link>
@@ -65,6 +64,6 @@
   <xacro:macro name="friction" params="link">
     <gazebo reference="${link}">
-      <mu1>0.5</mu1>
-      <mu2>0.5</mu2>
+      <mu1>0.2</mu1>
+      <mu2>0.2</mu2>
     </gazebo>
   </xacro:macro>

File: robots/tiger/urdf/v1/link.urdf.xacro (robot description, xacro)
@@ -19,5 +19,5 @@
     <xacro:damping_factor link="joint_junction_link${self}"/>
     <joint name="joint${self}_pitch" type="revolute">
-      <limit effort="6.6" lower="-1.57" upper="1.57" velocity="3.0"/>
+      <limit effort="100" lower="${-pi/2}" upper="${pi/2}" velocity="3.0"/>
       <parent link="joint_junction_link${self}"/>
       <child link="${child}"/>
@@ -28,5 +28,5 @@
     <xacro:joint_transmission joint="joint${self}_pitch"/>
     <xacro:if value="${leg == 1}">
-      <xacro:extra_module name="joint_junction_leg${self}" parent="joint_junction_link${self}" visible="1" collision="0" model_url="package://tiger/urdf/v1/mesh/leg/leg.dae">
+      <xacro:extra_module name="joint_junction_leg${self}" parent="joint_junction_link${self}" visible="1" collision="1" model_url="package://tiger/urdf/v1/mesh/leg/leg.dae">
         <origin xyz="0 0 -0.0283" rpy="0 ${pi} 0"/>
         <inertial>
@@ -86,5 +86,5 @@
     #### joints ####
     <joint name="joint${child1}_yaw" type="revolute">
-      <limit effort="6.6" lower="-1.57" upper="1.57" velocity="3.0"/>
+      <limit effort="100" lower="${-pi/2}" upper="${pi/2}" velocity="3.0"/>
       <parent link="center_link"/>
       <child link="joint_junction_link${child1}"/>
@@ -94,5 +94,5 @@
     </joint>
     <joint name="joint${child2}_yaw" type="revolute">
-      <limit effort="6.6" lower="-1.57" upper="1.57" velocity="3.0"/>
+      <limit effort="100" lower="${-pi/2}" upper="${pi/2}" velocity="3.0"/>
       <parent link="center_link"/>
       <child link="joint_junction_link${child2}"/>
@@ -102,5 +102,5 @@
     </joint>
     <joint name="joint${child3}_yaw" type="revolute">
-      <limit effort="6.6" lower="-1.57" upper="1.57" velocity="3.0"/>
+      <limit effort="100" lower="${-pi/2}" upper="${pi/2}" velocity="3.0"/>
       <parent link="center_link"/>
       <child link="joint_junction_link${child3}"/>
@@ -110,5 +110,5 @@
     </joint>
     <joint name="joint${child4}_yaw" type="revolute">
-      <limit effort="6.6" lower="-1.57" upper="1.57" velocity="3.0"/>
+      <limit effort="100" lower="${-pi/2}" upper="${pi/2}" velocity="3.0"/>
       <parent link="center_link"/>
       <child link="joint_junction_link${child4}"/>
@@ -161,6 +161,9 @@
         <mass value="0.2749981"/>
         <origin xyz="0.0145839 -0.0007152 -0.0219046" rpy="0 0 0"/>
-        <inertia
-            ixx="0.0004558" iyy="0.0005038" izz="0.0001566"
+        <!-- <inertia -->
+        <!--     ixx="0.0004558" iyy="0.0005038" izz="0.0001566" -->
+        <!--     ixy="0.0000029" iyz="-0.0000086" ixz="-0.0001245" /> -->
+        <inertia
+            ixx="0.004558" iyy="0.005038" izz="0.001566"
             ixy="0.0000029" iyz="-0.0000086" ixz="-0.0001245" />
       </inertial>
@@ -176,6 +179,9 @@
         <mass value="0.4336874"/>
         <origin xyz="0.0015167 0.0000151 -0.0010897" rpy="0 0 0"/>
-        <inertia
-            ixx="0.0004013" iyy="0.0075949" izz="0.0077808"
+        <!-- <inertia -->
+        <!--     ixx="0.0004013" iyy="0.0075949" izz="0.0077808" -->
+        <!--     ixy="0.0000001" iyz="-0.0000001" ixz="-0.0000103" /> -->
+        <inertia
+            ixx="0.004013" iyy="0.0075949" izz="0.0077808"
             ixy="0.0000001" iyz="-0.0000001" ixz="-0.0000103" />
       </inertial>
@@ -197,4 +203,37 @@
     </link>
     <xacro:damping_factor link="thrust${self}"/>
+    #### special part of duct fun ####
+    <joint name="edf${self}_left_mount" type="fixed">
+      <child link="edf${self}_left"/>
+      <parent link="gimbal_pitch_link${self}"/>
+      <origin rpy="0 0 0" xyz="0.15 0 0 "/>
+      <axis xyz="0 0 1"/>
+    </joint>
+    <link name="edf${self}_left">
+      <inertial>
+        <origin xyz="0 0 0" rpy="0 0 0"/>
+        <mass value="0.00001"/>
+        <inertia
+            ixx="0.000001" ixy="0.0" ixz="0.0"
+            iyy="0.000001" iyz="0.0"
+            izz="0.000002"/>
+      </inertial>
+    </link>
+    <joint name="edf${self}_right_mount" type="fixed">
+      <child link="edf${self}_right"/>
+      <parent link="gimbal_pitch_link${self}"/>
+      <origin rpy="0 0 0" xyz="-0.15 0 0 "/>
+      <axis xyz="0 0 1"/>
+    </joint>
+    <link name="edf${self}_right">
+      <inertial>
+        <origin xyz="0 0 0" rpy="0 0 0"/>
+        <mass value="0.00001"/>
+        <inertia
+            ixx="0.000001" ixy="0.0" ixz="0.0"
+            iyy="0.000001" iyz="0.0"
+            izz="0.000002"/>
+      </inertial>
+    </link>
     #### joint junction ####
     <xacro:unless value="${self == child}">
@@ -205,5 +244,5 @@
     <xacro:unless value="${self == child}">
       <joint name="joint${child}_yaw" type="revolute">
-        <limit effort="6.6" lower="${-pi / 2}" upper="${pi / 2}" velocity="3.0"/>
+        <limit effort="100" lower="${-pi/2}" upper="${pi}" velocity="3.0"/>
         <parent link="link${self}"/>
         <child link="joint_junction_link${child}"/>
@@ -214,5 +253,5 @@
     </xacro:unless>
     #### gimbal joint ####
-    <joint name="gimbal_roll${self}" type="continuous">
+    <joint name="gimbal${self}_roll" type="continuous">
       <limit effort="1.5" lower="${pi * -6}" upper="${pi * 6}" velocity="10.0"/>
       <parent link="link${self}"/>
@@ -222,10 +261,10 @@
       <dynamics damping="0.8" friction="0.0"/>
     </joint>
-    <joint name="gimbal_pitch${self}" type="continuous">
+    <joint name="gimbal${self}_pitch" type="continuous">
       <limit effort="1.5" lower="${pi * -6}" upper="${pi * 6}" velocity="10.0"/>
       <parent link="gimbal_roll_link${self}"/>
       <child link="gimbal_pitch_link${self}"/>
       <origin rpy="0 0 ${-pi / 2}" xyz="-0.0065 0.0 -0.027"/>
-      <axis xyz="1 0 0"/>
+      <axis xyz="-1 0 0"/>
       <dynamics damping="0.8" friction="0.0"/>
     </joint>
@@ -255,5 +294,5 @@
     <xacro:if value="${leg == 1}">
       <xacro:if value="${link_type == 'end'}">
-        <xacro:extra_module name="end_leg${self}" parent="link${self}" visible="1" collision="0"
+        <xacro:extra_module name="end_leg${self}" parent="link${self}" visible="1" collision="1"
                             model_url="package://tiger/urdf/v1/mesh/leg/end_leg.dae">
           <origin xyz="0.4835 0.0 0.0" rpy="0 0 0"/>
@@ -272,6 +311,6 @@
       <xacro:joint_transmission joint="joint${child}_yaw"/>
     </xacro:unless>
-    <xacro:joint_transmission joint="gimbal_roll${self}"/>
-    <xacro:joint_transmission joint="gimbal_pitch${self}"/>
+    <xacro:joint_transmission joint="gimbal${self}_roll"/>
+    <xacro:joint_transmission joint="gimbal${self}_pitch"/>
     <transmission name="rotor_tran${self}">
       <type>transmission_interface/SimpleTransmission</type>
