Commit message: [tiger] modify mesh and urdf

File: robots/tiger/robots/octo/v1_default/robot.urdf.xacro (robot description, xacro)
@@ -5,13 +5,23 @@
   <xacro:tiger_v1/>
   #### flight controller ####
-  <!-- TODO -->
-  <xacro:extra_module name = "fc" parent = "center_link" visible = "0">
-    <origin xyz="0 0 0" rpy="0 0 0"/>
+  <xacro:extra_module name = "fc" parent = "center_link" visible = "1"
+                      model_url = "package://tiger/urdf/v1/mesh/board/spinal.dae">
+    <origin xyz="-0.0129 0.0044 0.0398284" rpy="0 0 0"/>
     <inertial>
-      <origin xyz="0 0 0" rpy="0 0 0"/>
-      <mass value="0.001"/>
+      <mass value="0.0354160"/>
+      <origin xyz="0.0128576 0.0044678 -0.0226530" rpy="0 0 0"/>
       <inertia
-          ixx="0.000004" iyy="0.000004" izz="0.000008"
-          ixy="0.000001" ixz="-0.000001" iyz="-0.000000"/>
+          ixx="0.0000225" iyy="0.0000225" izz="0.0000346"
+          ixy="-0.0000001" iyz="0.0000000" ixz="0.0000000" />
+    </inertial>
+  </xacro:extra_module>
+  <xacro:extra_module name = "pc" parent = "center_link" visible = "0">
+    <origin xyz="0 0.089888 0.002" rpy="${pi/2} 0 0"/>
+    <inertial>
+      <mass value="0.1411331"/>
+      <origin xyz="0.0008915 0.0304136 0.0271590" rpy="0 0 0"/>
+      <inertia
+          ixx="0.0000768" iyy="0.0001380" izz="0.0001493"
+          ixy="0.0000018" iyz="0.0000071" ixz="-0.0000024" />
     </inertial>
   </xacro:extra_module>

File: robots/tiger/urdf/v1/common.xacro (robot description, xacro)
@@ -3,5 +3,5 @@
     xmlns:xacro="http://www.ros.org/wiki/xacro" name="tiger_common" >
   <!-- kinematics [m] -->
-  <xacro:property name="general_link_length" value="0.51661"/>
+  <xacro:property name="general_link_length" value="0.523"/>
   <xacro:property name="general_link_radius" value="0.025"/>
   <xacro:property name="center_link_radius" value="0.169"/>

File: robots/tiger/urdf/v1/link.urdf.xacro (robot description, xacro)
@@ -3,16 +3,30 @@
     xmlns:xacro="http://www.ros.org/wiki/xacro" name="tiger_link">
   <xacro:include filename="$(find tiger)/urdf/v1/common.xacro" />
-  <xacro:macro name="tiger_joint_junction_link" params="self child leg">
+  <xacro:macro name="tiger_joint_junction_link" params="self child leg type">
     <link name="joint_junction_link${self}">
-      <inertial>
-        <mass value="0.0953384"/>
-        <origin xyz="0.0257500 -0.0037552 0.0037552" rpy="0 0 0"/>
-        <inertia
-            ixx="0.0000741" iyy="0.0000792" izz="0.0000792"
-            ixy="-0.0000092" iyz="0.0000013" ixz="-0.0000092"/>
-      </inertial>
-      <xacro:mesh_model type="link/joint_junction_link">
-        <origin xyz="0 0 0" rpy="0 0 0"/>
-      </xacro:mesh_model>
+      <xacro:if value="${type == 'belt'}">
+        <inertial>
+          <mass value="0.0953384"/>
+          <origin xyz="0.0257500 -0.0037552 -0.0037552" rpy="0 0 0"/>
+          <inertia
+              ixx="0.0000741" iyy="0.0000792" izz="0.0000792"
+              ixy="-0.0000092" iyz="-0.0000013" ixz="0.0000092"/>
+        </inertial>
+        <xacro:mesh_model type="link/joint_junction_link_belt">
+          <origin xyz="0 0 0" rpy="0 0 0"/>
+        </xacro:mesh_model>
+      </xacro:if>
+      <xacro:if value="${type == 'wire_belt'}">
+        <inertial>
+          <mass value="0.1088219"/>
+          <origin xyz="0.0290910 -0.0078920 -0.0032913" rpy="0 0 0"/>
+          <inertia
+              ixx="0.0000906" iyy="0.0000939" izz="0.0001044"
+              ixy="-0.0000199" iyz="-0.0000028" ixz="0.0000104"/>
+        </inertial>
+        <xacro:mesh_model type="link/joint_junction_link_wire_belt">
+          <origin xyz="0 0 0" rpy="0 0 0"/>
+        </xacro:mesh_model>
+      </xacro:if>
     </link>
     <xacro:friction link="joint_junction_link${self}"/>
@@ -29,8 +43,8 @@
     <xacro:if value="${leg == 1}">
       <xacro:extra_module name="joint_junction_leg${self}" parent="joint_junction_link${self}" visible="1" collision="1" model_url="package://tiger/urdf/v1/mesh/leg/leg.dae">
-        <origin xyz="0 0 -0.0283" rpy="0 ${pi} 0"/>
+        <origin xyz="0 0 -0.0323" rpy="0 0 ${pi/2}"/>
         <inertial>
           <mass value="0.0230696"/>
-          <origin xyz="0 0.0000465 0.0474391" rpy="0 0 0"/>
+          <origin xyz="0 0.0000465 -0.0474391" rpy="0 0 0"/>
           <inertia
               ixx="0.0000295" iyy="0.0000293" izz="0.0000014"
@@ -62,9 +76,9 @@
     <link name="center_link">
       <inertial>
-        <mass value="1.1716010"/>
-        <origin xyz="0.0000000 0.0001441 0.0025981" rpy="0 0 0"/>
-        <inertia
-            ixx="0.0094720" iyy="0.0094643" izz="0.0170567"
-            ixy="-0.000000" ixz="-0.000000" iyz="-0.0000004"/>
+        <mass value="1.1780349"/>
+        <origin xyz="0.0000000 0.0001434 -0.0335345" rpy="0 0 0"/>
+        <inertia
+            ixx="0.0095261" iyy="0.0095185" izz="0.0171496"
+            ixy="0.0000000" iyz="0.0000057" ixz="0.0000000" />
       </inertial>
       <xacro:mesh_model type="link/center_link">
@@ -80,8 +94,8 @@
     <xacro:friction link="center_link"/>
     <xacro:damping_factor link="center_link"/>
-    <xacro:tiger_joint_junction_link self="${child1}" child="link${child1}" leg="${leg}"/>
-    <xacro:tiger_joint_junction_link self="${child2}" child="link${child2}" leg="${leg}"/>
-    <xacro:tiger_joint_junction_link self="${child3}" child="link${child3}" leg="${leg}"/>
-    <xacro:tiger_joint_junction_link self="${child4}" child="link${child4}" leg="${leg}"/>
+    <xacro:tiger_joint_junction_link self="${child1}" child="link${child1}" leg="${leg}" type="wire_belt"/>
+    <xacro:tiger_joint_junction_link self="${child2}" child="link${child2}" leg="${leg}" type="wire_belt"/>
+    <xacro:tiger_joint_junction_link self="${child3}" child="link${child3}" leg="${leg}" type="wire_belt"/>
+    <xacro:tiger_joint_junction_link self="${child4}" child="link${child4}" leg="${leg}" type="wire_belt"/>
     #### joints ####
     <joint name="joint${child1}_yaw" type="revolute">
@@ -89,5 +103,5 @@
       <parent link="center_link"/>
       <child link="joint_junction_link${child1}"/>
-      <origin rpy="0 0 ${pi / 4}" xyz="0.1195 0.1195 -0.0155"/>
+      <origin rpy="0 0 ${pi / 4}" xyz="0.12233 0.12233 -0.0155"/>
       <axis xyz="0 0 1"/>
       <dynamics damping="0.8" friction="0.0"/>
@@ -97,5 +111,5 @@
       <parent link="center_link"/>
       <child link="joint_junction_link${child2}"/>
-      <origin rpy="0 0 ${pi * 3 / 4}" xyz="-0.1195 0.1195 -0.0155"/>
+      <origin rpy="0 0 ${pi * 3 / 4}" xyz="-0.12233 0.12233 -0.0155"/>
       <axis xyz="0 0 1"/>
       <dynamics damping="0.8" friction="0.0"/>
@@ -105,5 +119,5 @@
       <parent link="center_link"/>
       <child link="joint_junction_link${child3}"/>
-      <origin rpy="0 0 ${pi * 5 / 4}" xyz="-0.1195 -0.1195 -0.0155"/>
+      <origin rpy="0 0 ${pi * 5 / 4}" xyz="-0.12233 -0.12233 -0.0155"/>
       <axis xyz="0 0 1"/>
       <dynamics damping="0.8" friction="0.0"/>
@@ -113,5 +127,5 @@
       <parent link="center_link"/>
       <child link="joint_junction_link${child4}"/>
-      <origin rpy="0 0 ${pi * 7 / 4}" xyz="0.1195 -0.1195 -0.0155"/>
+      <origin rpy="0 0 ${pi * 7 / 4}" xyz="0.12233 -0.12233 -0.0155"/>
       <axis xyz="0 0 1"/>
       <dynamics damping="0.8" friction="0.0"/>
@@ -129,9 +143,9 @@
       <xacro:if value="${link_type == 'general'}">
         <inertial>
-          <mass value="0.5104648"/>
-          <origin xyz="0.2574944 -0.0101285 0.0100891" rpy="0 0 0"/>
-          <inertia
-              ixx="0.0005824" iyy="0.0208863" izz="0.0208885"
-              ixy="0.0011182" iyz="0.0000521" ixz="0.0012028"/>
+          <mass value="0.5202337"/>
+          <origin xyz="0.2591013 -0.0021859 -0.0040686" rpy="0 0 0"/>
+          <inertia
+              ixx="0.0005100" iyy="0.0205461" izz="0.0201920"
+              ixy="0.0002263" iyz="-0.0000463" ixz="-0.0018418" />
         </inertial>
         <xacro:mesh_model type="link/general_link">
@@ -142,9 +156,9 @@
       <xacro:if value="${link_type == 'end'}">
         <inertial>
-          <mass value="0.3371341"/>
-          <origin xyz="0.1511545 -0.0153166 0.0000464" rpy="0 0 0"/>
-          <inertia
-              ixx="0.0002704" iyy="0.0079527" izz="0.0081722"
-              ixy="0.0005706" iyz="0.0000002" ixz="0.0000009" />
+          <mass value="0.3506780"/>
+          <origin xyz="0.1499167 -0.0148762 -0.0003693" rpy="0 0 0"/>
+          <inertia
+              ixx="0.0002771" iyy="0.0080082" izz="0.0082303"
+              ixy="0.0005694" iyz="-0.0000020" ixz="0.0000041" />
         </inertial>
         <xacro:mesh_model type="link/end_link">
@@ -165,5 +179,5 @@
         <!--     ixy="0.0000029" iyz="-0.0000086" ixz="-0.0001245" /> -->
         <inertia
-            ixx="0.004558" iyy="0.005038" izz="0.001566"
+            ixx="0.004558" iyy="0.0005038" izz="0.0001566"
             ixy="0.0000029" iyz="-0.0000086" ixz="-0.0001245" />
       </inertial>
@@ -177,12 +191,12 @@
     <link name="gimbal_pitch_link${self}">
       <inertial>
-        <mass value="0.4336874"/>
-        <origin xyz="0.0015167 0.0000151 -0.0010897" rpy="0 0 0"/>
+        <mass value="0.4335536"/>
+        <origin xyz="0.0000111 -0.0015087 -0.0010901" rpy="0 0 0"/>
         <!-- <inertia -->
-        <!--     ixx="0.0004013" iyy="0.0075949" izz="0.0077808" -->
-        <!--     ixy="0.0000001" iyz="-0.0000001" ixz="-0.0000103" /> -->
-        <inertia
-            ixx="0.004013" iyy="0.0075949" izz="0.0077808"
-            ixy="0.0000001" iyz="-0.0000001" ixz="-0.0000103" />
+        <!-- ixx="0.0075948" iyy="0.0004013" izz="0.0077807" -->
+        <!-- ixy="-0.0000001" iyz="0.0000103" ixz="-0.0000001" /> -->
+        <inertia
+            ixx="0.0075948" iyy="0.004013" izz="0.0077807"
+            ixy="-0.0000001" iyz="0.0000103" ixz="-0.0000001" />
       </inertial>
       <xacro:mesh_model type="link/pitch_link">
@@ -203,9 +217,9 @@
     </link>
     <xacro:damping_factor link="thrust${self}"/>
-    #### special part of duct fun ####
+    #### special part of duct fun (temporary)####
     <joint name="edf${self}_left_mount" type="fixed">
       <child link="edf${self}_left"/>
       <parent link="gimbal_pitch_link${self}"/>
-      <origin rpy="0 0 0" xyz="0.15 0 0 "/>
+      <origin rpy="0 0 0" xyz="0.1335 0 0 "/>
       <axis xyz="0 0 1"/>
     </joint>
@@ -223,5 +237,5 @@
       <child link="edf${self}_right"/>
       <parent link="gimbal_pitch_link${self}"/>
-      <origin rpy="0 0 0" xyz="-0.15 0 0 "/>
+      <origin rpy="0 0 0" xyz="-0.1335 0 0 "/>
       <axis xyz="0 0 1"/>
     </joint>
@@ -238,5 +252,5 @@
     #### joint junction ####
     <xacro:unless value="${self == child}">
-      <xacro:tiger_joint_junction_link self="${child}" child="link${child}" leg="${leg}"/>
+      <xacro:tiger_joint_junction_link self="${child}" child="link${child}" leg="${leg}" type="belt"/>
     </xacro:unless>
     #### joints ####
@@ -265,6 +279,6 @@
       <parent link="gimbal_roll_link${self}"/>
       <child link="gimbal_pitch_link${self}"/>
-      <origin rpy="0 0 ${-pi / 2}" xyz="-0.0065 0.0 -0.027"/>
-      <axis xyz="-1 0 0"/>
+      <origin rpy="0 0 0" xyz="-0.0065 0.0 -0.027"/>
+      <axis xyz="0 1 0"/>
       <dynamics damping="0.8" friction="0.0"/>
     </joint>
@@ -287,5 +301,5 @@
           <inertia
               ixx="0.0000994" iyy="0.0007104" izz="0.0006865"
-              ixy="0.0000000" iyz="0.0000000" ixz="-0.0000042"/>
+              ixy="0.0000000" iyz="0.0000000" ixz="-0.0000042" />
         </inertial>
       </xacro:extra_module>
@@ -298,9 +312,9 @@
           <origin xyz="0.4835 0.0 0.0" rpy="0 0 0"/>
           <inertial>
-            <mass value="0.0547396"/>
-            <origin xyz="0.0000000 -0.0000209 -0.0336847" rpy="0 0 0"/>
+            <mass value="0.0549856"/>
+            <origin xyz="0.0000000 -0.0000209 -0.0347870" rpy="0 0 0"/>
             <inertia
-                ixx="0.0001080" iyy="0.0001062" izz="0.0000123"
-                ixy="0.0000000" iyz="0.0000000" ixz="0.0000000"/>
+                ixx="0.0001158" iyy="0.0001141" izz="0.0000123"
+                ixy="0.0000000" iyz="0.0000000" ixz="0.0000000" />
           </inertial>
         </xacro:extra_module>

Commit message: [tiger] fix wrong fc position

File: robots/tiger/robots/octo/v1_default/robot.urdf.xacro (robot description, xacro)
@@ -7,5 +7,5 @@
   <xacro:extra_module name = "fc" parent = "center_link" visible = "1"
                       model_url = "package://tiger/urdf/v1/mesh/board/spinal.dae">
-    <origin xyz="-0.0129 0.0044 0.0398284" rpy="0 0 0"/>
+    <origin xyz="-0.0129 -0.0044 0.0398284" rpy="0 0 0"/>
     <inertial>
       <mass value="0.0354160"/>
