Commit message: [Dragon] 1. modify the control paramters.  - larger I term for xy position control  - faster gimbal roll speed for vertical link rotation case. 2. temporary change in the collision model for valve turning in gazebo.

File: robots/dragon/urdf/dragon_common.xacro (robot description, xacro)
@@ -24,5 +24,5 @@
     <origin rpy="0 0 0" xyz="${link_length* 0.5} 0 0"/>
     <geometry>
-    <box size="${link_length} 0.15 0.1686"/>
+    <box size="${link_length * 0.9} 0.05 0.1686"/>
     </geometry>
     </collision>
