Commit message: Update the urdf model for dragon, which uses LiHV battery

File: robots/dragon/urdf/dragon_link.urdf.xacro (robot description, xacro)
@@ -9,4 +9,10 @@
       <xacro:if value="${self == 1}">
         <inertial>
+          <origin xyz="${link_length* 0.5 + 15.09 * 0.001} ${-6.67 * 0.001} ${-27.21 * 0.001}" rpy="0 0 0"/>
+          <mass value="0.7968" />
+          <inertia
+              ixx="0.00095" iyy="0.0151" izz="0.0148"
+              ixy="-0.00098" ixz="0.0003" iyz="0.0001"/>
+          <!--
           <origin xyz="${link_length* 0.5 + 18.25 * 0.001} ${-7.17 * 0.001} ${-25.73 * 0.001}" rpy="0 0 0"/>
           <mass value="0.7408" />
@@ -14,4 +20,5 @@
               ixx="0.00095" iyy="0.0143" izz="0.0139"
               ixy="-0.00099" ixz="0.0003" iyz="0.0001"/>
+          -->
         </inertial>
         <xacro:link_model type="head_link" />
@@ -21,4 +28,10 @@
         <xacro:if value="${self == child}">
           <inertial>
+            <origin xyz="${link_length* 0.5 - 44.26 * 0.001} ${-0.11 * 0.001} ${-20.72 * 0.001}" rpy="0 0 0"/>
+            <mass value="0.7943" />
+            <inertia
+                ixx="0.0012" iyy="0.0145" izz="0.0134"
+                ixy="0.0" ixz="0.0003" iyz="0.0000"/>
+            <!--
             <origin xyz="${link_length* 0.5 - 45.44 * 0.001} ${-0.12 * 0.001} ${-18.74 * 0.001}" rpy="0 0 0"/>
             <mass value="0.7383" />
@@ -26,4 +39,5 @@
                 ixx="0.0012" iyy="0.0137" izz="0.0126"
                 ixy="0.0" ixz="0.0002" iyz="0.0"/>
+            -->
           </inertial>
           <xacro:link_model type="end_link" />
@@ -33,4 +47,10 @@
           <xacro:if value="${baselink}">
             <inertial>
+              <origin xyz="${link_length* 0.5 + 9.54 * 0.001} ${-4.74 * 0.001} ${-15.68 * 0.001}" rpy="0 0 0"/>
+              <mass value="1.1348" />
+              <inertia
+                  ixx="0.0018" iyy="0.0228" izz="0.0219"
+                  ixy="-0.0009" ixz="-0.0006" iyz="0.0001"/>
+              <!--
               <origin xyz="${link_length* 0.5 + 11.92 * 0.001} ${-4.98 * 0.001} ${-14.07 * 0.001}" rpy="0 0 0"/>
               <mass value="1.07879" />
@@ -38,4 +58,5 @@
                   ixx="0.0018" iyy="0.0219" izz="0.0211"
                   ixy="-0.001" ixz="-0.0007" iyz="0.0001"/>
+              -->
             </inertial>
             <xacro:link_model type="baselink" />
@@ -44,4 +65,10 @@
           <xacro:unless value="${baselink}">
             <inertial>
+              <origin xyz="${link_length* 0.5 - 12.78 * 0.001} ${-5.80 * 0.001} ${-16.95 * 0.001}" rpy="0 0 0"/>
+              <mass value="0.9289" />
+              <inertia
+                  ixx="0.0015" iyy="0.0198" izz="0.0189"
+                  ixy="-0.0008" ixz="-0.0001" iyz="0.0001"/>
+              <!--
               <origin xyz="${link_length* 0.5 - 11.75 * 0.001} ${-6.17 * 0.001} ${-15.04 * 0.001}" rpy="0 0 0"/>
               <mass value="0.8729" />
@@ -49,4 +76,5 @@
                   ixx="0.0015" iyy="0.0189" izz="0.0181"
                   ixy="-0.0008" ixz="-0.0002" iyz="0.0001"/>
+              -->
             </inertial>
             <xacro:link_model type="general_link" />

Commit message: [Dragon] implement rotor active winding action for dragon model, which allows the rotor stop thrust generation during winding. Also, modify the limits for gimbal roll angle in URDF to enable winding in gazebo.

File: robots/dragon/urdf/dragon_link.urdf.xacro (robot description, xacro)
@@ -86,5 +86,5 @@
     <!-- gimbal roll -->
     <joint name="gimbal${self}_roll" type="revolute">
-      <limit effort="3" lower="-3.14" upper="3.14" velocity="12.5"/>
+      <limit effort="3" lower="${-2*pi}" upper="${2*pi}" velocity="12.5"/>
       <parent link="link${self}"/>
       <child link="gimbal${self}_roll_module"/>
@@ -125,5 +125,5 @@
     <!-- gimbal pitch -->
     <joint name="gimbal${self}_pitch" type="revolute">
-      <limit effort="3" lower="-3.14" upper="3.14" velocity="12.5"/>
+      <limit effort="3" lower="${-2*pi}" upper="${2*pi}" velocity="12.5"/>
       <parent link="gimbal${self}_roll_module"/>
       <child link="gimbal${self}_pitch_module"/>

Commit message: [Dragon][URDF] enable link module without gimbal module

File: robots/dragon/urdf/dragon_link.urdf.xacro (robot description, xacro)
@@ -3,5 +3,5 @@
     xmlns:xacro="http://www.ros.org/wiki/xacro" name="dragon_link" >
   <!-- D-H kai description(different from prof.nakamura) -->
-  <xacro:macro name="dragon_module" params="self child baselink">
+  <xacro:macro name="dragon_module" params="self child baselink gimbal:=true">
     <!-- link -->
     <link name="link${self}">
@@ -84,119 +84,121 @@
     </link>
     <xacro:damping_factor link ="link${self}"/>
-    <!-- gimbal roll -->
-    <joint name="gimbal${self}_roll" type="revolute">
-      <limit effort="3" lower="-3.14" upper="3.14" velocity="12.5"/>
-      <parent link="link${self}"/>
-      <child link="gimbal${self}_roll_module"/>
-      <origin rpy="0 0 0" xyz="${link_length/2} 0 0"/>
-      <axis xyz="1 0 0"/>
-      <dynamics damping="0.1" friction="0.0"/>
-    </joint>
-    <link name="gimbal${self}_roll_module">
-      <inertial>
-        <origin xyz="${gimbal_roll_x_offset - 17.60 * 0.001} ${0.42 * 0.001} ${15.48 * 0.001}" rpy="0 0 0"/>
-        <mass value="0.4604" />
-        <inertia
-            ixx="0.0004" iyy="0.0004" izz="0.0003"
-            ixy="0" ixz="-0.0003" iyz="0"/>
-      </inertial>
-      <visual>
-        <origin xyz="${gimbal_roll_x_offset} 0 0" rpy="0 0 0"/>
-        <geometry>
-          <mesh filename="package://dragon/urdf/mesh/ducted_fan_gimbal_roll.dae"/>
-        </geometry>
-      </visual>
-      <!-- box collision not work good for FCL
-      <collision>
-        <origin rpy="0 0 0" xyz="${gimbal_roll_x_offset}  0 0"/>
-        <geometry>
-          <box size="0.1 0.3 0.1686"/>
-        </geometry>
-      </collision>
-      -->
-      <!-- cylinder collision geometry works well for FCL -->
-      <collision>
-        <origin rpy="${pi/2} 0 0" xyz="0 0 0.02"/>
-        <geometry>
-          <cylinder length="0.3" radius="0.09" />
-        </geometry>
-      </collision>
-    </link>
-    <!-- gimbal pitch -->
-    <joint name="gimbal${self}_pitch" type="revolute">
-      <limit effort="3" lower="-3.14" upper="3.14" velocity="12.5"/>
-      <parent link="gimbal${self}_roll_module"/>
-      <child link="gimbal${self}_pitch_module"/>
-      <origin rpy="0 0 0" xyz="0 0 ${gimbal_pitch_z_offset}"/>
-      <axis xyz="0 1 0"/>
-      <dynamics damping="0.1" friction="0.0"/>
-    </joint>
-    <link name="gimbal${self}_pitch_module">
-      <inertial>
-        <origin xyz="0 ${0.33 * 0.001}  ${-8.71 * 0.001}" rpy="0 0 0"/>
-        <mass value="0.5301" />
-        <inertia
-            ixx="0.0061" iyy="0.0001" izz="0.0061"
-            ixy="0.0" ixz="0.0" iyz="0.0"/>
-      </inertial>
-      <visual>
-        <origin xyz="0 0 0" rpy="0 0 0"/>
-        <geometry>
-          <mesh filename="package://dragon/urdf/mesh/ducted_fan_gimbal_pitch.dae"/>
-        </geometry>
-      </visual>
-    </link>
-    <!-- rotor -->
-    <joint name="rotor${self}" type="continuous">
-      <limit effort="100.0" lower="${min_force}" upper="${max_force}" velocity="0.5"/>
-      <parent link="gimbal${self}_pitch_module"/>
-      <child link="thrust${self}"/>
-      <origin rpy="0 0 0" xyz="0 0 0"/>
-      <axis xyz="0 0 1"/>
-    </joint>
-    <link name="thrust${self}">
-      <inertial>
-        <origin xyz="0 0 0" rpy="0 0 0"/>
-        <mass value="0.0001"/>
-        <inertia
-            ixx="0.00001" ixy="0.0" ixz="0.0"
-            iyy="0.00001" iyz="0.0"
-            izz="0.00002"/>
-      </inertial>
-    </link>
-    <!-- special part of duct fun -->
-    <joint name="edf${self}_left_mount" type="fixed">
-      <child link="edf${self}_left"/>
-      <parent link="gimbal${self}_pitch_module"/>
-      <origin rpy="0 0 0" xyz="0 0.1115 0 "/>
-      <axis xyz="0 0 1"/>
-    </joint>
-    <link name="edf${self}_left">
-      <inertial>
-        <origin xyz="0 0 0" rpy="0 0 0"/>
-        <mass value="0.00001"/>
-        <inertia
-            ixx="0.000001" ixy="0.0" ixz="0.0"
-            iyy="0.000001" iyz="0.0"
-            izz="0.000002"/>
-      </inertial>
-    </link>
-    <joint name="edf${self}_right_mount" type="fixed">
-      <child link="edf${self}_right"/>
-      <parent link="gimbal${self}_pitch_module"/>
-      <origin rpy="0 0 0" xyz="0 -0.1115 0 "/>
-      <axis xyz="0 0 1"/>
-    </joint>
-    <link name="edf${self}_right">
-      <inertial>
-        <origin xyz="0 0 0" rpy="0 0 0"/>
-        <mass value="0.00001"/>
-        <inertia
-            ixx="0.000001" ixy="0.0" ixz="0.0"
-            iyy="0.000001" iyz="0.0"
-            izz="0.000002"/>
-      </inertial>
-    </link>
-    <xacro:damping_factor link ="thrust${self}"/>
+    <xacro:if value="${gimbal}">
+      <!-- gimbal roll -->
+      <joint name="gimbal${self}_roll" type="revolute">
+        <limit effort="3" lower="-3.14" upper="3.14" velocity="12.5"/>
+        <parent link="link${self}"/>
+        <child link="gimbal${self}_roll_module"/>
+        <origin rpy="0 0 0" xyz="${link_length/2} 0 0"/>
+        <axis xyz="1 0 0"/>
+        <dynamics damping="0.1" friction="0.0"/>
+      </joint>
+      <link name="gimbal${self}_roll_module">
+        <inertial>
+          <origin xyz="${gimbal_roll_x_offset - 17.60 * 0.001} ${0.42 * 0.001} ${15.48 * 0.001}" rpy="0 0 0"/>
+          <mass value="0.4604" />
+          <inertia
+              ixx="0.0004" iyy="0.0004" izz="0.0003"
+              ixy="0" ixz="-0.0003" iyz="0"/>
+        </inertial>
+        <visual>
+          <origin xyz="${gimbal_roll_x_offset} 0 0" rpy="0 0 0"/>
+          <geometry>
+            <mesh filename="package://dragon/urdf/mesh/ducted_fan_gimbal_roll.dae"/>
+          </geometry>
+        </visual>
+        <!-- box collision not work good for FCL
+             <collision>
+             <origin rpy="0 0 0" xyz="${gimbal_roll_x_offset}  0 0"/>
+             <geometry>
+             <box size="0.1 0.3 0.1686"/>
+             </geometry>
+             </collision>
+        -->
+        <!-- cylinder collision geometry works well for FCL -->
+        <collision>
+          <origin rpy="${pi/2} 0 0" xyz="0 0 0.02"/>
+          <geometry>
+            <cylinder length="0.3" radius="0.09" />
+          </geometry>
+        </collision>
+      </link>
+      <!-- gimbal pitch -->
+      <joint name="gimbal${self}_pitch" type="revolute">
+        <limit effort="3" lower="-3.14" upper="3.14" velocity="12.5"/>
+        <parent link="gimbal${self}_roll_module"/>
+        <child link="gimbal${self}_pitch_module"/>
+        <origin rpy="0 0 0" xyz="0 0 ${gimbal_pitch_z_offset}"/>
+        <axis xyz="0 1 0"/>
+        <dynamics damping="0.1" friction="0.0"/>
+      </joint>
+      <link name="gimbal${self}_pitch_module">
+        <inertial>
+          <origin xyz="0 ${0.33 * 0.001}  ${-8.71 * 0.001}" rpy="0 0 0"/>
+          <mass value="0.5301" />
+          <inertia
+              ixx="0.0061" iyy="0.0001" izz="0.0061"
+              ixy="0.0" ixz="0.0" iyz="0.0"/>
+        </inertial>
+        <visual>
+          <origin xyz="0 0 0" rpy="0 0 0"/>
+          <geometry>
+            <mesh filename="package://dragon/urdf/mesh/ducted_fan_gimbal_pitch.dae"/>
+          </geometry>
+        </visual>
+      </link>
+      <!-- rotor -->
+      <joint name="rotor${self}" type="continuous">
+        <limit effort="100.0" lower="${min_force}" upper="${max_force}" velocity="0.5"/>
+        <parent link="gimbal${self}_pitch_module"/>
+        <child link="thrust${self}"/>
+        <origin rpy="0 0 0" xyz="0 0 0"/>
+        <axis xyz="0 0 1"/>
+      </joint>
+      <link name="thrust${self}">
+        <inertial>
+          <origin xyz="0 0 0" rpy="0 0 0"/>
+          <mass value="0.0001"/>
+          <inertia
+              ixx="0.00001" ixy="0.0" ixz="0.0"
+              iyy="0.00001" iyz="0.0"
+              izz="0.00002"/>
+        </inertial>
+      </link>
+      <!-- special part of duct fun -->
+      <joint name="edf${self}_left_mount" type="fixed">
+        <child link="edf${self}_left"/>
+        <parent link="gimbal${self}_pitch_module"/>
+        <origin rpy="0 0 0" xyz="0 0.1115 0 "/>
+        <axis xyz="0 0 1"/>
+      </joint>
+      <link name="edf${self}_left">
+        <inertial>
+          <origin xyz="0 0 0" rpy="0 0 0"/>
+          <mass value="0.00001"/>
+          <inertia
+              ixx="0.000001" ixy="0.0" ixz="0.0"
+              iyy="0.000001" iyz="0.0"
+              izz="0.000002"/>
+        </inertial>
+      </link>
+      <joint name="edf${self}_right_mount" type="fixed">
+        <child link="edf${self}_right"/>
+        <parent link="gimbal${self}_pitch_module"/>
+        <origin rpy="0 0 0" xyz="0 -0.1115 0 "/>
+        <axis xyz="0 0 1"/>
+      </joint>
+      <link name="edf${self}_right">
+        <inertial>
+          <origin xyz="0 0 0" rpy="0 0 0"/>
+          <mass value="0.00001"/>
+          <inertia
+              ixx="0.000001" ixy="0.0" ixz="0.0"
+              iyy="0.000001" iyz="0.0"
+              izz="0.000002"/>
+        </inertial>
+      </link>
+      <xacro:damping_factor link ="thrust${self}"/>
+    </xacro:if>
     <!-- joint -->
     <xacro:unless value="${self == child}">
@@ -304,34 +306,36 @@
       </transmission>
     </xacro:unless>
-    <transmission name="gimbal${self}_roll_tran">
-      <type>transmission_interface/SimpleTransmission</type>
-      <joint name="gimbal${self}_roll">
-        <hardwareInterface>hardware_interface/EffortJointInterface</hardwareInterface>
-      </joint>
-      <actuator name="gimbal_servo{self}_roll">
-        <hardwareInterface>hardware_interface/EffortJointInterface</hardwareInterface>
-        <mechanicalReduction>1</mechanicalReduction>
-      </actuator>
-    </transmission>
-    <transmission name="gimbal${self}_pitch_tran">
-      <type>transmission_interface/SimpleTransmission</type>
-      <joint name="gimbal${self}_pitch">
-        <hardwareInterface>hardware_interface/EffortJointInterface</hardwareInterface>
-      </joint>
-      <actuator name="gimbal_servo{self}_pitch">
-        <hardwareInterface>hardware_interface/EffortJointInterface</hardwareInterface>
-        <mechanicalReduction>1</mechanicalReduction>
-      </actuator>
-    </transmission>
-    <transmission name="rotor${self}_tran">
-      <type>transmission_interface/SimpleTransmission</type>
-      <joint name="rotor${self}">
-        <hardwareInterface>RotorInterface</hardwareInterface>
-      </joint>
-      <actuator name="rotor${self}">
-        <hardwareInterface>RotorInterface</hardwareInterface>
-        <mechanicalReduction>1</mechanicalReduction>
-      </actuator>
-      </transmission>
+    <xacro:if value="${gimbal}">
+      <transmission name="gimbal${self}_roll_tran">
+        <type>transmission_interface/SimpleTransmission</type>
+        <joint name="gimbal${self}_roll">
+          <hardwareInterface>hardware_interface/EffortJointInterface</hardwareInterface>
+        </joint>
+        <actuator name="gimbal_servo{self}_roll">
+          <hardwareInterface>hardware_interface/EffortJointInterface</hardwareInterface>
+          <mechanicalReduction>1</mechanicalReduction>
+        </actuator>
+      </transmission>
+      <transmission name="gimbal${self}_pitch_tran">
+        <type>transmission_interface/SimpleTransmission</type>
+        <joint name="gimbal${self}_pitch">
+          <hardwareInterface>hardware_interface/EffortJointInterface</hardwareInterface>
+        </joint>
+        <actuator name="gimbal_servo{self}_pitch">
+          <hardwareInterface>hardware_interface/EffortJointInterface</hardwareInterface>
+          <mechanicalReduction>1</mechanicalReduction>
+        </actuator>
+      </transmission>
+      <transmission name="rotor${self}_tran">
+        <type>transmission_interface/SimpleTransmission</type>
+        <joint name="rotor${self}">
+          <hardwareInterface>RotorInterface</hardwareInterface>
+        </joint>
+        <actuator name="rotor${self}">
+          <hardwareInterface>RotorInterface</hardwareInterface>
+          <mechanicalReduction>1</mechanicalReduction>
+        </actuator>
+      </transmission>
+    </xacro:if>
     <xacro:friction self ="${self}"/>
   </xacro:macro>

Commit message: [Dragon][Perching Arm] enable to put the gimbal to the head of a link and create the robot model of perching arm

File: robots/dragon/urdf/dragon_link.urdf.xacro (robot description, xacro)
@@ -3,5 +3,5 @@
     xmlns:xacro="http://www.ros.org/wiki/xacro" name="dragon_link" >
   <!-- D-H kai description(different from prof.nakamura) -->
-  <xacro:macro name="dragon_module" params="self child baselink gimbal:=true">
+  <xacro:macro name="dragon_module" params="self child baselink gimbal:=true head_gimbal:=false">
     <!-- link -->
     <link name="link${self}">
@@ -90,5 +90,10 @@
         <parent link="link${self}"/>
         <child link="gimbal${self}_roll_module"/>
-        <origin rpy="0 0 0" xyz="${link_length/2} 0 0"/>
+        <xacro:if value="${head_gimbal}">
+          <origin rpy="0 0 0" xyz="0.05 0 0"/>
+        </xacro:if>
+        <xacro:unless value="${head_gimbal}">
+          <origin rpy="0 0 0" xyz="${link_length/2} 0 0"/>
+        </xacro:unless>
         <axis xyz="1 0 0"/>
         <dynamics damping="0.1" friction="0.0"/>

Commit message: [Dragon][VIM4] refactor the system to use Khadas VIM4

File: robots/dragon/urdf/dragon_link.urdf.xacro (robot description, xacro)
@@ -47,9 +47,9 @@
           <xacro:if value="${baselink}">
             <inertial>
-              <origin xyz="${link_length* 0.5 + 9.54 * 0.001} ${-4.74 * 0.001} ${-15.68 * 0.001}" rpy="0 0 0"/>
-              <mass value="1.1348" />
+              <origin xyz="${link_length* 0.5 + 2.23 * 0.001} ${-5.59 * 0.001} ${-14.86 * 0.001}" rpy="0 0 0"/>
+              <mass value="1.055" />
               <inertia
-                  ixx="0.0018" iyy="0.0228" izz="0.0219"
-                  ixy="-0.0009" ixz="-0.0006" iyz="0.0001"/>
+                  ixx="0.0016" iyy="0.0221" izz="0.0213"
+                  ixy="-0.0009" ixz="-0.0002" iyz="-0.0001"/>
               <!--
               <origin xyz="${link_length* 0.5 + 11.92 * 0.001} ${-4.98 * 0.001} ${-14.07 * 0.001}" rpy="0 0 0"/>
