Commit message: [tiger] improve urdf

File: robots/tiger/urdf/v1/common.xacro (robot description, xacro)
@@ -8,5 +8,6 @@
   <xacro:property name="center_link_height" value="0.0928"/>
   <!-- dynamics -->
-  <xacro:property name="max_force" value="36"/> <!-- [N] -->
+  <xacro:property name="max_force" value="36"/> ### [N]
+  <xacro:property name="max_joint_torque" value="6.6"/>  ### [N]
   <xacro:macro name="mesh_model" params="type *origin">
     <visual>

File: robots/tiger/urdf/v1/link.urdf.xacro (robot description, xacro)
@@ -19,5 +19,5 @@
     <xacro:damping_factor link="joint_junction_link${self}"/>
     <joint name="joint${self}_pitch" type="revolute">
-      <limit effort="100" lower="${-pi/2}" upper="${pi/2}" velocity="3.0"/>
+      <limit effort="${max_joint_torque}" lower="${-pi/2}" upper="${pi/2}" velocity="3.0"/>
       <parent link="joint_junction_link${self}"/>
       <child link="${child}"/>
@@ -86,5 +86,5 @@
     #### joints ####
     <joint name="joint${child1}_yaw" type="revolute">
-      <limit effort="100" lower="${-pi/2}" upper="${pi/2}" velocity="3.0"/>
+      <limit effort="${max_joint_torque}" lower="${-pi/2}" upper="${pi/2}" velocity="3.0"/>
       <parent link="center_link"/>
       <child link="joint_junction_link${child1}"/>
@@ -94,5 +94,5 @@
     </joint>
     <joint name="joint${child2}_yaw" type="revolute">
-      <limit effort="100" lower="${-pi/2}" upper="${pi/2}" velocity="3.0"/>
+      <limit effort="${max_joint_torque}" lower="${-pi/2}" upper="${pi/2}" velocity="3.0"/>
       <parent link="center_link"/>
       <child link="joint_junction_link${child2}"/>
@@ -102,5 +102,5 @@
     </joint>
     <joint name="joint${child3}_yaw" type="revolute">
-      <limit effort="100" lower="${-pi/2}" upper="${pi/2}" velocity="3.0"/>
+      <limit effort="${max_joint_torque}" lower="${-pi/2}" upper="${pi/2}" velocity="3.0"/>
       <parent link="center_link"/>
       <child link="joint_junction_link${child3}"/>
@@ -110,5 +110,5 @@
     </joint>
     <joint name="joint${child4}_yaw" type="revolute">
-      <limit effort="100" lower="${-pi/2}" upper="${pi/2}" velocity="3.0"/>
+      <limit effort="${max_joint_torque}" lower="${-pi/2}" upper="${pi/2}" velocity="3.0"/>
       <parent link="center_link"/>
       <child link="joint_junction_link${child4}"/>
@@ -244,5 +244,5 @@
     <xacro:unless value="${self == child}">
       <joint name="joint${child}_yaw" type="revolute">
-        <limit effort="100" lower="${-pi/2}" upper="${pi}" velocity="3.0"/>
+        <limit effort="${max_joint_torque}" lower="${-pi/2}" upper="${pi}" velocity="3.0"/>
         <parent link="link${self}"/>
         <child link="joint_junction_link${child}"/>

Commit message: [tiger] modify leg collision model

File: robots/tiger/urdf/v1/common.xacro (robot description, xacro)
@@ -7,4 +7,7 @@
   <xacro:property name="center_link_radius" value="0.169"/>
   <xacro:property name="center_link_height" value="0.0928"/>
+  <xacro:property name="leg_radius" value="0.01"/>
+  <xacro:property name="leg_length" value="0.1005"/>
+  <xacro:property name="end_leg_length" value="0.1325"/>
   <!-- dynamics -->
   <xacro:property name="max_force" value="36"/> ### [N]
@@ -26,4 +29,20 @@
       <geometry>
         <cylinder radius="${general_link_radius}" length="${general_link_length}"/>
+      </geometry>
+    </collision>
+  </xacro:macro>
+  <xacro:macro name="leg_collision_model">
+    <collision>
+      <origin xyz="0 0 ${leg_length * -0.5}" rpy="0 0 0"/>
+      <geometry>
+        <cylinder radius="${leg_radius}" length="${leg_length}"/>
+      </geometry>
+    </collision>
+  </xacro:macro>
+  <xacro:macro name="end_leg_collision_model">
+    <collision>
+      <origin xyz="0 0 ${end_leg_length * -0.5}" rpy="0 0 0"/>
+      <geometry>
+        <cylinder radius="${leg_radius}" length="${end_leg_length}"/>
       </geometry>
     </collision>
@@ -53,4 +72,22 @@
     </link>
   </xacro:macro>
+  <xacro:macro name="extra_module_with_collision" params="name parent *origin *inertial *collision visible:=0 model_url:=0">
+    <joint name="${parent}2${name}" type="fixed">
+      <parent link="${parent}"/>
+      <child link="${name}"/>
+      <xacro:insert_block name="origin" />
+    </joint>
+    <link name="${name}">
+      <xacro:insert_block name="inertial" />
+      <xacro:if value="${visible == 1}">
+        <visual>
+          <geometry>
+            <mesh filename="${model_url}"/>
+          </geometry>
+        </visual>
+      </xacro:if>
+      <xacro:insert_block name="collision"/>
+    </link>
+  </xacro:macro>
   <xacro:macro name="joint_transmission" params="joint">
     <transmission name="{joint}_tran">

File: robots/tiger/urdf/v1/link.urdf.xacro (robot description, xacro)
@@ -42,5 +42,5 @@
     <xacro:joint_transmission joint="joint${self}_pitch"/>
     <xacro:if value="${leg == 1}">
-      <xacro:extra_module name="joint_junction_leg${self}" parent="joint_junction_link${self}" visible="1" collision="1" model_url="package://tiger/urdf/v1/mesh/leg/leg.dae">
+      <xacro:extra_module_with_collision name="joint_junction_leg${self}" parent="joint_junction_link${self}" visible="1" model_url="package://tiger/urdf/v1/mesh/leg/leg.dae">
         <origin xyz="0 0 -0.0323" rpy="0 0 ${pi/2}"/>
         <inertial>
@@ -51,5 +51,6 @@
               ixy="0.0000000" iyz="0.0000000" ixz="0.0000000"/>
         </inertial>
-      </xacro:extra_module>
+        <xacro:leg_collision_model/>
+      </xacro:extra_module_with_collision>
     </xacro:if>
   </xacro:macro>
@@ -305,8 +306,8 @@
       </xacro:extra_module>
     </xacro:if>
-    #### leg ####
+    #### end leg ####
     <xacro:if value="${leg == 1}">
       <xacro:if value="${link_type == 'end'}">
-        <xacro:extra_module name="end_leg${self}" parent="link${self}" visible="1" collision="1"
+        <xacro:extra_module_with_collision name="end_leg${self}" parent="link${self}" visible="1"
                             model_url="package://tiger/urdf/v1/mesh/leg/end_leg.dae">
           <origin xyz="0.4835 0.0 0.0" rpy="0 0 0"/>
@@ -318,5 +319,6 @@
                 ixy="0.0000000" iyz="0.0000000" ixz="0.0000000" />
           </inertial>
-        </xacro:extra_module>
+          <xacro:end_leg_collision_model/>
+        </xacro:extra_module_with_collision>
       </xacro:if>
     </xacro:if>

Commit message: [Tiger] refactor the urdf model to be compatible for dragon full_vectoring control

File: robots/tiger/urdf/v1/common.xacro (robot description, xacro)
@@ -13,4 +13,5 @@
   <xacro:property name="max_force" value="36"/> ### [N]
   <xacro:property name="max_joint_torque" value="6.6"/>  ### [N]
+  <xacro:property name="max_joint_vel" value="0.1"/>  ### [N]
   <baselink name="fc" />
   <thrust_link name="thrust" />

File: robots/tiger/urdf/v1/link.urdf.xacro (robot description, xacro)
@@ -33,5 +33,5 @@
     <xacro:damping_factor link="joint_junction_link${self}"/>
     <joint name="joint${self}_pitch" type="revolute">
-      <limit effort="${max_joint_torque}" lower="${-pi/2}" upper="${pi/2}" velocity="3.0"/>
+      <limit effort="${max_joint_torque}" lower="${-pi/2}" upper="${pi/2}" velocity="${max_joint_vel}"/>
       <parent link="joint_junction_link${self}"/>
       <child link="${child}"/>
@@ -101,5 +101,5 @@
     #### joints ####
     <joint name="joint${child1}_yaw" type="revolute">
-      <limit effort="${max_joint_torque}" lower="${-pi/2}" upper="${pi/2}" velocity="3.0"/>
+      <limit effort="${max_joint_torque}" lower="${-pi/2}" upper="${pi/2}" velocity="${max_joint_vel}"/>
       <parent link="center_link"/>
       <child link="joint_junction_link${child1}"/>
@@ -109,5 +109,5 @@
     </joint>
     <joint name="joint${child2}_yaw" type="revolute">
-      <limit effort="${max_joint_torque}" lower="${-pi/2}" upper="${pi/2}" velocity="3.0"/>
+      <limit effort="${max_joint_torque}" lower="${-pi/2}" upper="${pi/2}" velocity="${max_joint_vel}"/>
       <parent link="center_link"/>
       <child link="joint_junction_link${child2}"/>
@@ -117,5 +117,5 @@
     </joint>
     <joint name="joint${child3}_yaw" type="revolute">
-      <limit effort="${max_joint_torque}" lower="${-pi/2}" upper="${pi/2}" velocity="3.0"/>
+      <limit effort="${max_joint_torque}" lower="${-pi/2}" upper="${pi/2}" velocity="${max_joint_vel}"/>
       <parent link="center_link"/>
       <child link="joint_junction_link${child3}"/>
@@ -125,5 +125,5 @@
     </joint>
     <joint name="joint${child4}_yaw" type="revolute">
-      <limit effort="${max_joint_torque}" lower="${-pi/2}" upper="${pi/2}" velocity="3.0"/>
+      <limit effort="${max_joint_torque}" lower="${-pi/2}" upper="${pi/2}" velocity="${max_joint_vel}"/>
       <parent link="center_link"/>
       <child link="joint_junction_link${child4}"/>
@@ -172,5 +172,5 @@
     <xacro:damping_factor link="link${self}"/>
     #### gimbal roll ####
-    <link name="gimbal_roll_link${self}">
+    <link name="gimbal${self}_roll_module">
       <inertial>
         <mass value="0.2749981"/>
@@ -187,8 +187,8 @@
       </xacro:mesh_model>
     </link>
-    <xacro:friction link="gimbal_roll_link${self}"/>
-    <xacro:damping_factor link="gimbal_roll_link${self}"/>
+    <xacro:friction link="gimbal${self}_roll_module"/>
+    <xacro:damping_factor link="gimbal${self}_roll_module"/>
     #### gimbal pitch ####
-    <link name="gimbal_pitch_link${self}">
+    <link name="gimbal${self}_pitch_module">
       <inertial>
         <mass value="0.4335536"/>
@@ -205,6 +205,6 @@
       </xacro:mesh_model>
     </link>
-    <xacro:friction link="gimbal_pitch_link${self}"/>
-    <xacro:damping_factor link="gimbal_pitch_link${self}"/>
+    <xacro:friction link="gimbal${self}_pitch_module"/>
+    <xacro:damping_factor link="gimbal${self}_pitch_module"/>
     #### thrust link (virtual) ####
     <link name="thrust${self}">
@@ -221,5 +221,5 @@
     <joint name="edf${self}_left_mount" type="fixed">
       <child link="edf${self}_left"/>
-      <parent link="gimbal_pitch_link${self}"/>
+      <parent link="gimbal${self}_pitch_module"/>
       <origin rpy="0 0 0" xyz="0.1335 0 0 "/>
       <axis xyz="0 0 1"/>
@@ -237,5 +237,5 @@
     <joint name="edf${self}_right_mount" type="fixed">
       <child link="edf${self}_right"/>
-      <parent link="gimbal_pitch_link${self}"/>
+      <parent link="gimbal${self}_pitch_module"/>
       <origin rpy="0 0 0" xyz="-0.1335 0 0 "/>
       <axis xyz="0 0 1"/>
@@ -259,5 +259,5 @@
     <xacro:unless value="${self == child}">
       <joint name="joint${child}_yaw" type="revolute">
-        <limit effort="${max_joint_torque}" lower="${-pi/2}" upper="${pi}" velocity="3.0"/>
+        <limit effort="${max_joint_torque}" lower="${-pi/2}" upper="${pi}" velocity="${max_joint_vel}"/>
         <parent link="link${self}"/>
         <child link="joint_junction_link${child}"/>
@@ -271,5 +271,5 @@
       <limit effort="1.5" lower="${pi * -6}" upper="${pi * 6}" velocity="10.0"/>
       <parent link="link${self}"/>
-      <child link="gimbal_roll_link${self}"/>
+      <child link="gimbal${self}_roll_module"/>
       <origin rpy="0 0 0" xyz="0.268 0.0 0.0"/>
       <axis xyz="1 0 0"/>
@@ -278,6 +278,6 @@
     <joint name="gimbal${self}_pitch" type="continuous">
       <limit effort="1.5" lower="${pi * -6}" upper="${pi * 6}" velocity="10.0"/>
-      <parent link="gimbal_roll_link${self}"/>
-      <child link="gimbal_pitch_link${self}"/>
+      <parent link="gimbal${self}_roll_module"/>
+      <child link="gimbal${self}_pitch_module"/>
       <origin rpy="0 0 0" xyz="-0.0065 0.0 -0.027"/>
       <axis xyz="0 1 0"/>
@@ -287,5 +287,5 @@
     <joint name="rotor${self}" type="continuous">
      <limit effort="100.0" lower="0" upper="${max_force}" velocity="0.5"/>
-      <parent link="gimbal_pitch_link${self}"/>
+      <parent link="gimbal${self}_pitch_module"/>
       <child link="thrust${self}"/>
       <origin rpy="0 0 0" xyz="0 0 0"/>

Commit message: [Tiger] further update the robot model

File: robots/tiger/urdf/v1/common.xacro (robot description, xacro)
@@ -8,5 +8,5 @@
   <xacro:property name="center_link_height" value="0.0928"/>
   <xacro:property name="leg_radius" value="0.01"/>
-  <xacro:property name="leg_length" value="0.1005"/>
+  <xacro:property name="leg_length" value="0.1045"/>
   <xacro:property name="end_leg_length" value="0.1325"/>
   <!-- dynamics -->

File: robots/tiger/urdf/v1/link.urdf.xacro (robot description, xacro)
@@ -8,8 +8,8 @@
         <inertial>
           <mass value="0.095"/>
-          <origin xyz="0.026 -0.004 0.004" rpy="0 0 0"/>
+          <origin xyz="0.026 0.004 0.004" rpy="0 0 0"/>
           <inertia
               ixx="0.000074" iyy="0.000079" izz="0.000079"
-              ixy="-0.000009" iyz="0.000001" ixz="-0.000009"/>
+              ixy="0.000009" iyz="-0.000001" ixz="-0.000009"/>
         </inertial>
         <xacro:mesh_model type="link/joint_junction_link">
@@ -20,8 +20,8 @@
         <inertial>
           <mass value="0.103"/>
-          <origin xyz="0.028 -0.007 -0.003" rpy="0 0 0"/>
+          <origin xyz="0.028 0.007 0.003" rpy="0 0 0"/>
           <inertia
               ixx="0.000087" iyy="0.000087" izz="0.000096"
-              ixy="-0.000016" iyz="-0.000002" ixz="0.000010"/>
+              ixy="0.000016" iyz="-0.000002" ixz="-0.000010"/>
         </inertial>
         <xacro:mesh_model type="link/joint_junction_link_large_pitch_pulley">
@@ -54,9 +54,9 @@
     <xacro:joint_transmission joint="joint${self}_pitch"/>
     <xacro:if value="${leg == 1}">
-      <xacro:extra_module_with_collision name="joint_junction_leg${self}" parent="joint_junction_link${self}" visible="1" model_url="package://tiger/urdf/v1/mesh/leg/leg.dae">
-        <origin xyz="0 0 -0.0323" rpy="0 0 ${pi/2}"/>
-        <inertial>
-          <mass value="0.024"/>
-          <origin xyz="0 0 -0.047" rpy="0 0 0"/>
+      <xacro:extra_module_with_collision name="joint_junction_leg${self}" parent="joint_junction_link${self}" visible="1" model_url="package://tiger/urdf/v1/mesh/leg/long_leg.dae">
+        <origin xyz="0 0 -0.0283" rpy="0 0 ${pi/2}"/>
+        <inertial>
+          <mass value="0.027"/>
+          <origin xyz="0 0 -0.046" rpy="0 0 0"/>
           <inertia
               ixx="0.000029" iyy="0.000029" izz="0.000002"
@@ -90,8 +90,8 @@
       <inertial>
         <mass value="1.1780349"/>
-        <origin xyz="0.0000000 0.0001434 -0.0335345" rpy="0 0 0"/>
-        <inertia
-            ixx="0.0095261" iyy="0.0095185" izz="0.0171496"
-            ixy="0.0000000" iyz="0.0000057" ixz="0.0000000" />
+        <origin xyz="0.0 0.0 0.027" rpy="0 0 0"/>
+        <inertia
+            ixx="0.009512" iyy="0.009512" izz="0.017150"
+            ixy="0.000000" iyz="0.000000" ixz="0.000000" />
       </inertial>
       <xacro:mesh_model type="link/center_link">
@@ -157,8 +157,8 @@
         <inertial>
           <mass value="0.523"/>
-          <origin xyz="0.257 -0.002 0.017" rpy="0 0 0"/>
-          <inertia
-              ixx="0.000383" iyy="0.021153" izz="0.020931"
-              ixy="0.000250" iyz="-0.000021" ixz="0.000494" />
+          <origin xyz="0.257 -0.002 0.004" rpy="0 0 0"/>
+          <inertia
+              ixx="0.000519" iyy="0.021290" izz="0.020931"
+              ixy="-0.000246" iyz="-0.000044" ixz="0.001893" />
         </inertial>
         <xacro:mesh_model type="link/general_link">
@@ -170,8 +170,8 @@
         <inertial>
           <mass value="0.347"/>
-          <origin xyz="0.157 -0.015 0" rpy="0 0 0"/>
+          <origin xyz="0.157 0.015 0" rpy="0 0 0"/>
           <inertia
               ixx="0.000276" iyy="0.008551" izz="0.008772"
-              ixy="0.000606" iyz="-0.000002" ixz="-0.000029" />
+              ixy="-0.000606" iyz="0.000001" ixz="-0.000031" />
         </inertial>
         <xacro:mesh_model type="link/end_link">
@@ -317,5 +317,5 @@
         <xacro:extra_module_with_collision name="end_leg${self}" parent="link${self}" visible="1"
                             model_url="package://tiger/urdf/v1/mesh/leg/end_leg.dae">
-          <origin xyz="0.160 0.0 0.0" rpy="0 0 0"/>
+          <origin xyz="${0.160 + 0.335} 0.0 0.0" rpy="0 0 0"/>
           <inertial>
             <mass value="0.055"/>
