Commit message: [Tiger] implement thrust force allocation with consideration of joint torque for flight control

File: robots/tiger/urdf/v1/link.urdf.xacro (robot description, xacro)
@@ -296,5 +296,5 @@
       <xacro:extra_module name="bat${self}" parent="link${self}" visible="1"
                           model_url="package://tiger/urdf/v1/mesh/battery/ZIPPY-3000-25C-6S.dae">
-        <origin xyz="0.1395 0.0 -0.018" rpy="0 ${pi} 0"/>
+        <origin xyz="${0.1395 + 0.25} 0.0 -0.018" rpy="0 ${pi} 0"/>
         <inertial>
           <mass value="0.4170000"/>

Commit message: [Tiger] fix the wrong position of edf in urdf

File: robots/tiger/urdf/v1/link.urdf.xacro (robot description, xacro)
@@ -222,5 +222,5 @@
       <child link="edf${self}_left"/>
       <parent link="gimbal${self}_pitch_module"/>
-      <origin rpy="0 0 0" xyz="0.1335 0 0 "/>
+      <origin rpy="0 0 0" xyz="0 0.1335 0 "/>
       <axis xyz="0 0 1"/>
     </joint>
@@ -238,5 +238,5 @@
       <child link="edf${self}_right"/>
       <parent link="gimbal${self}_pitch_module"/>
-      <origin rpy="0 0 0" xyz="-0.1335 0 0 "/>
+      <origin rpy="0 0 0" xyz="0 -0.1335 0 "/>
       <axis xyz="0 0 1"/>
     </joint>

Commit message: [Tiger] update the robot model for tiger v1

File: robots/tiger/urdf/v1/link.urdf.xacro (robot description, xacro)
@@ -145,5 +145,5 @@
         <inertial>
           <mass value="0.5202337"/>
-          <origin xyz="0.2591013 -0.0021859 -0.0040686" rpy="0 0 0"/>
+          <origin xyz="0.2591013 -0.0021859 0.0040686" rpy="0 0 0"/>
           <inertia
               ixx="0.0005100" iyy="0.0205461" izz="0.0201920"
@@ -296,5 +296,5 @@
       <xacro:extra_module name="bat${self}" parent="link${self}" visible="1"
                           model_url="package://tiger/urdf/v1/mesh/battery/ZIPPY-3000-25C-6S.dae">
-        <origin xyz="${0.1395 + 0.25} 0.0 -0.018" rpy="0 ${pi} 0"/>
+        <origin xyz="${0.4} 0.0 -0.018" rpy="0 ${pi} 0"/>
         <inertial>
           <mass value="0.4170000"/>

Commit message: [Tiger] update the inerital parameters and the dynamics config for gazebo

File: robots/tiger/urdf/v1/link.urdf.xacro (robot description, xacro)
@@ -7,9 +7,9 @@
       <xacro:if value="${type == 'belt'}">
         <inertial>
-          <mass value="0.0953384"/>
-          <origin xyz="0.0257500 -0.0037552 -0.0037552" rpy="0 0 0"/>
-          <inertia
-              ixx="0.0000741" iyy="0.0000792" izz="0.0000792"
-              ixy="-0.0000092" iyz="-0.0000013" ixz="0.0000092"/>
+          <mass value="0.095"/>
+          <origin xyz="0.026 -0.004 0.004" rpy="0 0 0"/>
+          <inertia
+              ixx="0.000074" iyy="0.000079" izz="0.000079"
+              ixy="-0.000009" iyz="0.000001" ixz="-0.000009"/>
         </inertial>
         <xacro:mesh_model type="link/joint_junction_link_belt">
@@ -19,9 +19,9 @@
       <xacro:if value="${type == 'wire_belt'}">
         <inertial>
-          <mass value="0.1088219"/>
-          <origin xyz="0.0290910 -0.0078920 -0.0032913" rpy="0 0 0"/>
-          <inertia
-              ixx="0.0000906" iyy="0.0000939" izz="0.0001044"
-              ixy="-0.0000199" iyz="-0.0000028" ixz="0.0000104"/>
+          <mass value="0.103"/>
+          <origin xyz="0.028 -0.007 -0.003" rpy="0 0 0"/>
+          <inertia
+              ixx="0.000087" iyy="0.000087" izz="0.000096"
+              ixy="-0.000016" iyz="-0.000002" ixz="0.000010"/>
         </inertial>
         <xacro:mesh_model type="link/joint_junction_link_wire_belt">
@@ -38,5 +38,5 @@
       <origin rpy="0 0 0" xyz="0.0515 0.0 0.0"/>
       <axis xyz="0 1 0"/>
-      <dynamics damping="0.8" friction="0.0"/>
+      <dynamics damping="0.9" friction="0.0"/>
     </joint>
     <xacro:joint_transmission joint="joint${self}_pitch"/>
@@ -45,9 +45,9 @@
         <origin xyz="0 0 -0.0323" rpy="0 0 ${pi/2}"/>
         <inertial>
-          <mass value="0.0230696"/>
-          <origin xyz="0 0.0000465 -0.0474391" rpy="0 0 0"/>
-          <inertia
-              ixx="0.0000295" iyy="0.0000293" izz="0.0000014"
-              ixy="0.0000000" iyz="0.0000000" ixz="0.0000000"/>
+          <mass value="0.024"/>
+          <origin xyz="0 0 -0.047" rpy="0 0 0"/>
+          <inertia
+              ixx="0.000029" iyy="0.000029" izz="0.000002"
+              ixy="0.000000" iyz="0.000000" ixz="0.000000"/>
         </inertial>
         <xacro:leg_collision_model/>
@@ -106,5 +106,5 @@
       <origin rpy="0 0 ${pi / 4}" xyz="0.12233 0.12233 -0.0155"/>
       <axis xyz="0 0 1"/>
-      <dynamics damping="0.8" friction="0.0"/>
+      <dynamics damping="0.9" friction="0.0"/>
     </joint>
     <joint name="joint${child2}_yaw" type="revolute">
@@ -114,5 +114,5 @@
       <origin rpy="0 0 ${pi * 3 / 4}" xyz="-0.12233 0.12233 -0.0155"/>
       <axis xyz="0 0 1"/>
-      <dynamics damping="0.8" friction="0.0"/>
+      <dynamics damping="0.9" friction="0.0"/>
     </joint>
     <joint name="joint${child3}_yaw" type="revolute">
@@ -122,5 +122,5 @@
       <origin rpy="0 0 ${pi * 5 / 4}" xyz="-0.12233 -0.12233 -0.0155"/>
       <axis xyz="0 0 1"/>
-      <dynamics damping="0.8" friction="0.0"/>
+      <dynamics damping="0.9" friction="0.0"/>
     </joint>
     <joint name="joint${child4}_yaw" type="revolute">
@@ -130,5 +130,5 @@
       <origin rpy="0 0 ${pi * 7 / 4}" xyz="0.12233 -0.12233 -0.0155"/>
       <axis xyz="0 0 1"/>
-      <dynamics damping="0.8" friction="0.0"/>
+      <dynamics damping="0.9" friction="0.0"/>
     </joint>
     #### hardware interface ####
@@ -144,9 +144,9 @@
       <xacro:if value="${link_type == 'general'}">
         <inertial>
-          <mass value="0.5202337"/>
-          <origin xyz="0.2591013 -0.0021859 0.0040686" rpy="0 0 0"/>
-          <inertia
-              ixx="0.0005100" iyy="0.0205461" izz="0.0201920"
-              ixy="0.0002263" iyz="-0.0000463" ixz="-0.0018418" />
+          <mass value="0.523"/>
+          <origin xyz="0.257 -0.002 0.017" rpy="0 0 0"/>
+          <inertia
+              ixx="0.000383" iyy="0.021153" izz="0.020931"
+              ixy="0.000250" iyz="-0.000021" ixz="0.000494" />
         </inertial>
         <xacro:mesh_model type="link/general_link">
@@ -157,9 +157,9 @@
       <xacro:if value="${link_type == 'end'}">
         <inertial>
-          <mass value="0.3506780"/>
-          <origin xyz="0.1499167 -0.0148762 -0.0003693" rpy="0 0 0"/>
-          <inertia
-              ixx="0.0002771" iyy="0.0080082" izz="0.0082303"
-              ixy="0.0005694" iyz="-0.0000020" ixz="0.0000041" />
+          <mass value="0.347"/>
+          <origin xyz="0.157 -0.015 0" rpy="0 0 0"/>
+          <inertia
+              ixx="0.000276" iyy="0.008551" izz="0.008772"
+              ixy="0.000606" iyz="-0.000002" ixz="-0.000029" />
         </inertial>
         <xacro:mesh_model type="link/end_link">
@@ -174,12 +174,9 @@
     <link name="gimbal${self}_roll_module">
       <inertial>
-        <mass value="0.2749981"/>
+        <mass value="0.275"/>
         <origin xyz="0.0145839 -0.0007152 -0.0219046" rpy="0 0 0"/>
-        <!-- <inertia -->
-        <!--     ixx="0.0004558" iyy="0.0005038" izz="0.0001566" -->
-        <!--     ixy="0.0000029" iyz="-0.0000086" ixz="-0.0001245" /> -->
-        <inertia
-            ixx="0.004558" iyy="0.0005038" izz="0.0001566"
-            ixy="0.0000029" iyz="-0.0000086" ixz="-0.0001245" />
+        <inertia
+            ixx="0.000456" iyy="0.000504" izz="0.000157"
+            ixy="0.000003" iyz="-0.000009" ixz="-0.000125" />
       </inertial>
       <xacro:mesh_model type="link/roll_link">
@@ -192,12 +189,9 @@
     <link name="gimbal${self}_pitch_module">
       <inertial>
-        <mass value="0.4335536"/>
+        <mass value="0.434"/>
         <origin xyz="0.0000111 -0.0015087 -0.0010901" rpy="0 0 0"/>
-        <!-- <inertia -->
-        <!-- ixx="0.0075948" iyy="0.0004013" izz="0.0077807" -->
-        <!-- ixy="-0.0000001" iyz="0.0000103" ixz="-0.0000001" /> -->
-        <inertia
-            ixx="0.0075948" iyy="0.004013" izz="0.0077807"
-            ixy="-0.0000001" iyz="0.0000103" ixz="-0.0000001" />
+        <inertia
+            ixx="0.007595" iyy="0.000401" izz="0.007781"
+            ixy="0.000000" iyz="0.000010" ixz="0.000000" />
       </inertial>
       <xacro:mesh_model type="link/pitch_link">
@@ -264,5 +258,5 @@
         <origin rpy="0 0 0" xyz="${general_link_length} 0 0"/>
         <axis xyz="0 0 1"/>
-        <dynamics damping="0.8" friction="0.0"/>
+        <dynamics damping="0.9" friction="0.0"/>
       </joint>
     </xacro:unless>
@@ -274,5 +268,5 @@
       <origin rpy="0 0 0" xyz="0.268 0.0 0.0"/>
       <axis xyz="1 0 0"/>
-      <dynamics damping="0.8" friction="0.0"/>
+      <dynamics damping="0.1" friction="0.0"/>
     </joint>
     <joint name="gimbal${self}_pitch" type="continuous">
@@ -282,5 +276,5 @@
       <origin rpy="0 0 0" xyz="-0.0065 0.0 -0.027"/>
       <axis xyz="0 1 0"/>
-      <dynamics damping="0.8" friction="0.0"/>
+      <dynamics damping="0.1" friction="0.0"/>
     </joint>
     #### rotor joint (virtual) ####
@@ -296,11 +290,11 @@
       <xacro:extra_module name="bat${self}" parent="link${self}" visible="1"
                           model_url="package://tiger/urdf/v1/mesh/battery/ZIPPY-3000-25C-6S.dae">
-        <origin xyz="${0.4} 0.0 -0.018" rpy="0 ${pi} 0"/>
-        <inertial>
-          <mass value="0.4170000"/>
-          <origin xyz="-0.0005920 0.0000000 0.0211150" rpy="0 0 0"/>
-          <inertia
-              ixx="0.0000994" iyy="0.0007104" izz="0.0006865"
-              ixy="0.0000000" iyz="0.0000000" ixz="-0.0000042" />
+        <origin xyz="0.410 0.0 -0.039" rpy="${-pi/2} 0 0"/>
+        <inertial>
+          <mass value="0.417"/>
+          <origin xyz="-0.001 0.0 0.0" rpy="0 0 0"/>
+          <inertia
+              ixx="0.000099" iyy="0.000700" izz="0.000673"
+              ixy="0.000000" iyz="0.000000" ixz="-0.000001" />
         </inertial>
       </xacro:extra_module>
@@ -311,11 +305,11 @@
         <xacro:extra_module_with_collision name="end_leg${self}" parent="link${self}" visible="1"
                             model_url="package://tiger/urdf/v1/mesh/leg/end_leg.dae">
-          <origin xyz="0.4835 0.0 0.0" rpy="0 0 0"/>
+          <origin xyz="0.160 0.0 0.0" rpy="0 0 0"/>
           <inertial>
-            <mass value="0.0549856"/>
-            <origin xyz="0.0000000 -0.0000209 -0.0347870" rpy="0 0 0"/>
+            <mass value="0.055"/>
+            <origin xyz="0.0000000 0.0000 -0.035" rpy="0 0 0"/>
             <inertia
-                ixx="0.0001158" iyy="0.0001141" izz="0.0000123"
-                ixy="0.0000000" iyz="0.0000000" ixz="0.0000000" />
+                ixx="0.000116" iyy="0.000114" izz="0.000012"
+                ixy="0.000000" iyz="0.000000" ixz="0.000000" />
           </inertial>
           <xacro:end_leg_collision_model/>

Commit message: [Tiger] update the visual model

File: robots/tiger/urdf/v1/link.urdf.xacro (robot description, xacro)
@@ -13,9 +13,9 @@
               ixy="-0.000009" iyz="0.000001" ixz="-0.000009"/>
         </inertial>
-        <xacro:mesh_model type="link/joint_junction_link_belt">
-          <origin xyz="0 0 0" rpy="0 0 0"/>
-        </xacro:mesh_model>
-      </xacro:if>
-      <xacro:if value="${type == 'wire_belt'}">
+        <xacro:mesh_model type="link/joint_junction_link">
+          <origin xyz="0 0 0" rpy="0 0 0"/>
+        </xacro:mesh_model>
+      </xacro:if>
+      <xacro:if value="${type == 'large_pitch_pulley'}">
         <inertial>
           <mass value="0.103"/>
@@ -25,5 +25,17 @@
               ixy="-0.000016" iyz="-0.000002" ixz="0.000010"/>
         </inertial>
-        <xacro:mesh_model type="link/joint_junction_link_wire_belt">
+        <xacro:mesh_model type="link/joint_junction_link_large_pitch_pulley">
+          <origin xyz="0 0 0" rpy="0 0 0"/>
+        </xacro:mesh_model>
+      </xacro:if>
+      <xacro:if value="${type == 'wire'}">
+        <inertial>
+          <mass value="0.103"/>
+          <origin xyz="0.028 -0.007 -0.003" rpy="0 0 0"/>
+          <inertia
+              ixx="0.000087" iyy="0.000087" izz="0.000096"
+              ixy="-0.000016" iyz="-0.000002" ixz="0.000010"/>
+        </inertial>
+        <xacro:mesh_model type="link/joint_junction_link_wire">
           <origin xyz="0 0 0" rpy="0 0 0"/>
         </xacro:mesh_model>
@@ -95,8 +107,8 @@
     <xacro:friction link="center_link"/>
     <xacro:damping_factor link="center_link"/>
-    <xacro:tiger_joint_junction_link self="${child1}" child="link${child1}" leg="${leg}" type="wire_belt"/>
-    <xacro:tiger_joint_junction_link self="${child2}" child="link${child2}" leg="${leg}" type="wire_belt"/>
-    <xacro:tiger_joint_junction_link self="${child3}" child="link${child3}" leg="${leg}" type="wire_belt"/>
-    <xacro:tiger_joint_junction_link self="${child4}" child="link${child4}" leg="${leg}" type="wire_belt"/>
+    <xacro:tiger_joint_junction_link self="${child1}" child="link${child1}" leg="${leg}" type="large_pitch_pulley"/>
+    <xacro:tiger_joint_junction_link self="${child2}" child="link${child2}" leg="${leg}" type="large_pitch_pulley"/>
+    <xacro:tiger_joint_junction_link self="${child3}" child="link${child3}" leg="${leg}" type="large_pitch_pulley"/>
+    <xacro:tiger_joint_junction_link self="${child4}" child="link${child4}" leg="${leg}" type="large_pitch_pulley"/>
     #### joints ####
     <joint name="joint${child1}_yaw" type="revolute">

Commit message: [Tiger] further improve the position of battery in general link

File: robots/tiger/urdf/v1/link.urdf.xacro (robot description, xacro)
@@ -302,5 +302,10 @@
       <xacro:extra_module name="bat${self}" parent="link${self}" visible="1"
                           model_url="package://tiger/urdf/v1/mesh/battery/ZIPPY-3000-25C-6S.dae">
-        <origin xyz="0.410 0.0 -0.039" rpy="${-pi/2} 0 0"/>
+        <xacro:if value="${link_type == 'general'}">
+          <origin xyz="0.430 0.0 -0.039" rpy="${-pi/2} 0 0"/>
+        </xacro:if>
+        <xacro:if value="${link_type == 'end'}">
+          <origin xyz="0.410 0.0 -0.039" rpy="${-pi/2} 0 0"/>
+        </xacro:if>
         <inertial>
           <mass value="0.417"/>
