Commit message: [Mini Quadrotor] add urdf model for Realsense T265

File: robots/mini_quadrotor/urdf/robot.urdf.xacro (robot description, xacro)
@@ -118,5 +118,5 @@
   <!-- spinal -->
   <xacro:extra_module name = "fc" parent = "main_body" visible = "0" >
-    <origin xyz="0 0 0" rpy="0 0 0"/>
+    <origin xyz="-0.012 -0.003 0.023" rpy="0 0 0"/>
     <inertial>
       <mass value = "00" />
@@ -125,4 +125,17 @@
           ixx="0.0" ixy="0.0" ixz="0.0"
           iyy="0.0" iyz="0.0" izz="0.0"/>
+    </inertial>
+  </xacro:extra_module>
+  <!-- front realsense t265 -->
+  <xacro:extra_module name = "realsense_t265" parent = "main_body" visible = "1" scale= "1"
+                      model_url = "package://mini_quadrotor/urdf/mesh/realSense_t265.STL">
+    <origin xyz="0.1095 0.00775 0.0125" rpy="0 0 0"/>
+    <inertial>
+      <mass value = "0.07" />
+      <origin xyz="-0.007 -0.007 0" rpy="0 0 0"/>
+      <inertia
+          ixx="0.0" ixy="0.0" ixz="0.0"
+          iyy="0.0001" iyz="0.0"
+          izz="0.0001"/>
     </inertial>
   </xacro:extra_module>

Commit message: [Mini Quadrotor] update the model related to realsense t265

File: robots/mini_quadrotor/urdf/robot.urdf.xacro (robot description, xacro)
@@ -140,4 +140,15 @@
     </inertial>
   </xacro:extra_module>
+  <!-- pose frame for realsense t265 -->
+  <xacro:extra_module name = "realsense_pose_frame" parent = "realsense_t265" visible = "0" >
+    <origin xyz="-0.005 0.0 0.0" rpy="0 0 0"/>
+    <inertial>
+      <mass value = "0.0" />
+      <origin xyz="0 0 0" rpy="0 0 0"/>
+      <inertia
+          ixx="0.0" ixy="0.0" ixz="0.0"
+          iyy="0.0" iyz="0.0" izz="0.0"/>
+    </inertial>
+  </xacro:extra_module>
   <!-- battery -->
   <xacro:extra_module name = "battery" parent = "main_body" visible = "1" model_url = "package://mini_quadrotor/urdf/mesh/turnigy_3S_2200mAh.dae" >

Commit message: [Mini Quadrotor][WIP] create the quadrotor model with 3D LiDAR of Livox MID360

File: robots/mini_quadrotor/urdf/robot.urdf.xacro (robot description, xacro)
@@ -6,6 +6,6 @@
   <thrust_link name="thrust" />
   <!-- kinematics [m] -->
-  <xacro:property name="rotor_x" value="0.070" />
-  <xacro:property name="rotor_y" value="0.086" />
+  <xacro:property name="rotor_x" value="0.085" />
+  <xacro:property name="rotor_y" value="0.085" />
   <xacro:property name="rotor_z" value="0.026" />
   <!-- dynamics -->
@@ -96,15 +96,15 @@
   <link name="main_body">
     <inertial>
-      <mass value = "0.432" />
-      <origin xyz="0 0 0.017" rpy="0 0 0"/>
+      <mass value = "0.832" />
+      <origin xyz="0.002 0 ${0.028 - 0.002}" rpy="0 0 0"/> <!-- TODO: true cog pos -->
       <inertia
-          ixx="0.0021" ixy="0" ixz="0"
-          iyy="0.0015" iyz="0"
-          izz="0.0032"/>
+          ixx="0.0030" ixy="0" ixz="0"
+          iyy="0.0030" iyz="0"
+          izz="0.0045"/>
     </inertial>
     <visual>
       <origin rpy="0 0 0" xyz="0 0 0"/>
       <geometry>
-        <mesh filename="package://mini_quadrotor/urdf/mesh/main_body.dae" />
+        <mesh filename="package://mini_quadrotor/urdf/mesh/main_body_livox.dae" />
       </geometry>
     </visual>
@@ -128,21 +128,32 @@
   </xacro:extra_module>
   <!-- front realsense t265 -->
-  <xacro:extra_module name = "realsense_t265" parent = "main_body" visible = "1" scale= "1"
-                      model_url = "package://mini_quadrotor/urdf/mesh/realSense_t265.STL">
-    <origin xyz="0.1095 0.00775 0.0125" rpy="0 0 0"/>
+  <!-- <xacro:extra_module name = "realsense_t265" parent = "main_body" visible = "1" scale= "1" -->
+  <!--                     model_url = "package://mini_quadrotor/urdf/mesh/realSense_t265.STL"> -->
+  <!--   <origin xyz="0.1095 0.00775 0.0125" rpy="0 0 0"/> -->
+  <!--   <inertial> -->
+  <!--     <mass value = "0.07" /> -->
+  <!--     <origin xyz="-0.007 -0.007 0" rpy="0 0 0"/> -->
+  <!--     <inertia -->
+  <!--         ixx="0.0" ixy="0.0" ixz="0.0" -->
+  <!--         iyy="0.0001" iyz="0.0" -->
+  <!--         izz="0.0001"/> -->
+  <!--   </inertial> -->
+  <!-- </xacro:extra_module> -->
+  <!-- pose frame for realsense t265 -->
+  <!-- <xacro:extra_module name = "realsense_pose_frame" parent = "realsense_t265" visible = "0" > -->
+  <!--   <origin xyz="-0.005 0.0 0.0" rpy="0 0 0"/> -->
+  <!--   <inertial> -->
+  <!--     <mass value = "0.0" /> -->
+  <!--     <origin xyz="0 0 0" rpy="0 0 0"/> -->
+  <!--     <inertia -->
+  <!--         ixx="0.0" ixy="0.0" ixz="0.0" -->
+  <!--         iyy="0.0" iyz="0.0" izz="0.0"/> -->
+  <!--   </inertial> -->
+  <!-- </xacro:extra_module> -->
+  <!-- livox mid360 -->
+  <xacro:extra_module name = "lidar_imu" parent = "main_body" visible = "0" > <!-- should be IMU frame -->
+    <origin xyz="${0.011} ${0.02329} ${0.0425 + 0.047 - 0.04412}" rpy="0 0 0"/> <!-- TODO: the true pos -->
     <inertial>
-      <mass value = "0.07" />
-      <origin xyz="-0.007 -0.007 0" rpy="0 0 0"/>
-      <inertia
-          ixx="0.0" ixy="0.0" ixz="0.0"
-          iyy="0.0001" iyz="0.0"
-          izz="0.0001"/>
-    </inertial>
-  </xacro:extra_module>
-  <!-- pose frame for realsense t265 -->
-  <xacro:extra_module name = "realsense_pose_frame" parent = "realsense_t265" visible = "0" >
-    <origin xyz="-0.005 0.0 0.0" rpy="0 0 0"/>
-    <inertial>
-      <mass value = "0.0" />
+      <mass value = "00" />
       <origin xyz="0 0 0" rpy="0 0 0"/>
       <inertia
@@ -153,5 +164,5 @@
   <!-- battery -->
   <xacro:extra_module name = "battery" parent = "main_body" visible = "1" model_url = "package://mini_quadrotor/urdf/mesh/turnigy_3S_2200mAh.dae" >
-    <origin xyz="0.0105 0 -0.012" rpy="0 0 0"/>
+    <origin xyz="0.0 0 -0.035" rpy="${pi/2} 0 0"/>
     <inertial>
       <mass value = "0.188" />

Commit message: [Mini Quadrotor][WIP] create the quadrotor model with 3D LiDAR of Livox MID360

File: robots/mini_quadrotor/urdf/robot.urdf.xacro (robot description, xacro)
@@ -6,6 +6,6 @@
   <thrust_link name="thrust" />
   <!-- kinematics [m] -->
-  <xacro:property name="rotor_x" value="0.070" />
-  <xacro:property name="rotor_y" value="0.086" />
+  <xacro:property name="rotor_x" value="0.085" />
+  <xacro:property name="rotor_y" value="0.085" />
   <xacro:property name="rotor_z" value="0.026" />
   <!-- dynamics -->
@@ -96,15 +96,15 @@
   <link name="main_body">
     <inertial>
-      <mass value = "0.432" />
-      <origin xyz="0 0 0.017" rpy="0 0 0"/>
+      <mass value = "0.832" />
+      <origin xyz="0.002 0 ${0.028 - 0.002}" rpy="0 0 0"/> <!-- TODO: true cog pos -->
       <inertia
-          ixx="0.0021" ixy="0" ixz="0"
-          iyy="0.0015" iyz="0"
-          izz="0.0032"/>
+          ixx="0.0030" ixy="0" ixz="0"
+          iyy="0.0030" iyz="0"
+          izz="0.0045"/>
     </inertial>
     <visual>
       <origin rpy="0 0 0" xyz="0 0 0"/>
       <geometry>
-        <mesh filename="package://mini_quadrotor/urdf/mesh/main_body.dae" />
+        <mesh filename="package://mini_quadrotor/urdf/mesh/main_body_livox.dae" />
       </geometry>
     </visual>
@@ -127,7 +127,18 @@
     </inertial>
   </xacro:extra_module>
+  <!-- livox mid360 -->
+  <xacro:extra_module name = "lidar_imu" parent = "main_body" visible = "0" > <!-- should be IMU frame -->
+    <origin xyz="${0.011} ${0.02329} ${0.0425 + 0.047 - 0.04412}" rpy="0 0 0"/> <!-- TODO: the true pos -->
+    <inertial>
+      <mass value = "00" />
+      <origin xyz="0 0 0" rpy="0 0 0"/>
+      <inertia
+          ixx="0.0" ixy="0.0" ixz="0.0"
+          iyy="0.0" iyz="0.0" izz="0.0"/>
+    </inertial>
+  </xacro:extra_module>
   <!-- battery -->
   <xacro:extra_module name = "battery" parent = "main_body" visible = "1" model_url = "package://mini_quadrotor/urdf/mesh/turnigy_3S_2200mAh.dae" >
-    <origin xyz="0.0105 0 -0.012" rpy="0 0 0"/>
+    <origin xyz="0.0 0 -0.035" rpy="${pi/2} 0 0"/>
     <inertial>
       <mass value = "0.188" />

Commit message: [Mini Quadrotor][FAST LIO] update URDF to use spinal IMU for FAST LIO

File: robots/mini_quadrotor/urdf/robot.urdf.xacro (robot description, xacro)
@@ -118,5 +118,5 @@
   <!-- spinal -->
   <xacro:extra_module name = "fc" parent = "main_body" visible = "0" >
-    <origin xyz="0 0 0" rpy="0 0 0"/>
+    <origin xyz="-0.02 -0.005 0.03" rpy="0 0 0"/>
     <inertial>
       <mass value = "00" />
@@ -129,5 +129,5 @@
   <!-- livox mid360 -->
   <xacro:extra_module name = "lidar_imu" parent = "main_body" visible = "0" > <!-- should be IMU frame -->
-    <origin xyz="${0.011} ${0.02329} ${0.0425 + 0.047 - 0.04412}" rpy="0 0 0"/> <!-- TODO: the true pos -->
+    <origin xyz="0 0 0" rpy="0 0 0"/> <!-- TODO: the true pos -->
     <inertial>
       <mass value = "00" />

Commit message: [Mini Quadrotor] update the URDF with the CFRP 3D LiDAR protector

File: robots/mini_quadrotor/urdf/robot.urdf.xacro (robot description, xacro)
@@ -96,5 +96,5 @@
   <link name="main_body">
     <inertial>
-      <mass value = "0.832" />
+      <mass value = "0.860" />
       <origin xyz="0.002 0 ${0.028 - 0.002}" rpy="0 0 0"/> <!-- TODO: true cog pos -->
       <inertia

Commit message: [Mini Quadrotor][WIP] add usb camera module

File: robots/mini_quadrotor/urdf/robot.urdf.xacro (robot description, xacro)
@@ -149,4 +149,15 @@
     </inertial>
   </xacro:extra_module>
+  <!-- front usb camera -->
+  <xacro:extra_module name = "usb_cam" parent = "main_body" visible = "0"  >
+    <origin xyz="0.09 0 0" rpy="0 0 0"/>
+    <inertial>
+      <mass value = "0.02" />
+      <origin xyz="0 0 0" rpy="0 0 0"/>
+      <inertia
+          ixx="0.00001" ixy="0.0" ixz="0.0"
+          iyy="0.00001" iyz="0.0" izz="0.00002"/>
+    </inertial>
+  </xacro:extra_module>
   <!-- propellers -->
   <xacro:propeller_module id = "1" x = "${-rotor_x}" y = "${-rotor_y}" z = "${rotor_z}" direction = "-1" />
