Commit message: Squashed commits from origin/master with the following latest commit:
commit 7ac7184987f22b20589dec3767a93025762c6017
Merge: e11261e2 212c7171
Author: 趙　漠居(Zhao, Moju) <chou@jsk.imi.i.u-tokyo.ac.jp>
Date:   Mon Apr 15 09:57:03 2024 +0900

    Merge pull request #610 from sugikazu75/PR/package/depend

    [Package.xml] Resolve dependency to other package

File: robots/hydrus/urdf/link.urdf.xacro (robot description, xacro)
@@ -200,5 +200,5 @@
       </xacro:if>
       <xacro:unless value="${tilt_mode == 1}">
-        <origin rpy="0 0 0" xyz="${link_length* 0.5} 0 0"/>
+        <origin rpy="0 0 0" xyz="${link_length* 0.5} 0 0.013"/>
       </xacro:unless>
       <axis xyz="0 0 ${rotor_direction}"/>
@@ -220,4 +220,15 @@
         </geometry>
       </collision>
+      <visual>
+        <origin rpy="0 0 0" xyz="0 0 0.032"/>
+        <geometry>
+          <xacro:if value="${rotor_direction == 1}">
+            <mesh filename="package://hydrus/urdf/mesh/propeller/T-motor-CF-14inch-CCW.dae"/>
+          </xacro:if>
+          <xacro:if value="${rotor_direction == -1}">
+            <mesh filename="package://hydrus/urdf/mesh/propeller/T-motor-CF-14inch-CW.dae"/>
+          </xacro:if>
+        </geometry>
+      </visual>
     </link>
     <xacro:damping_factor link ="thrust${self}"/>

File: robots/hydrus_xi/robots/hex_branch/xavier201811.urdf.xacro (robot description, xacro)
@@ -22,6 +22,6 @@
       <mass value="0.549000"/>
       <inertia
-          ixx="-0.000452" iyy="-0.000453" izz="-0.000000"
-          ixy="0.000000" ixz="-0.000014" iyz="-0.000002"/>
+          ixx="0.000452" iyy="0.000453" izz="0.000453"
+          ixy="0.000000" ixz="0.00000" iyz="0.0000000"/>
     </inertial>
   </xacro:extra_module>

File: robots/hydrus_xi/urdf/branch_type_link.urdf.xacro (robot description, xacro)
@@ -172,4 +172,15 @@
             izz="${rotor_mass * .5 * rotor_radius * rotor_radius}"/>
       </inertial>
+      <visual>
+        <origin rpy="0 0 0" xyz="0 0 0"/>
+        <geometry>
+          <xacro:if value="${rotor_direction == 1}">
+            <mesh filename="package://hydrus_xi/urdf/mesh/propeller/T-motor-CF-14inch-CCW.dae"/>
+          </xacro:if>
+          <xacro:if value="${rotor_direction == -1}">
+            <mesh filename="package://hydrus_xi/urdf/mesh/propeller/T-motor-CF-14inch-CW.dae"/>
+          </xacro:if>
+        </geometry>
+      </visual>
     </link>
     <xacro:damping_factor link="thrust${self}"/>

File: robots/hydrus_xi/urdf/link.urdf.xacro (robot description, xacro)
@@ -88,4 +88,15 @@
             izz="${rotor_mass * .5 * rotor_radius * rotor_radius}"/>
       </inertial>
+      <visual>
+        <origin rpy="0 0 0" xyz="0 0 0.01"/>
+        <geometry>
+          <xacro:if value="${rotor_direction == 1}">
+            <mesh filename="package://hydrus_xi/urdf/mesh/propeller/T-motor-CF-14inch-CCW.dae"/>
+          </xacro:if>
+          <xacro:if value="${rotor_direction == -1}">
+            <mesh filename="package://hydrus_xi/urdf/mesh/propeller/T-motor-CF-14inch-CW.dae"/>
+          </xacro:if>
+        </geometry>
+      </visual>
     </link>
     <xacro:damping_factor link="thrust${self}"/>
