Commit message: [WIP] configuration for success hovering

File: robots/aero_mobility/urdf/robot.urdf.xacro (robot description, xacro)
@@ -102,5 +102,5 @@
   <link name="main_body">
     <inertial>
-      <mass value = "24.05" />
+      <mass value = "${24.05 - 2.6 * 4}" />
       <origin xyz="0 0 0" rpy="0 0 0"/>
       <inertia
@@ -124,5 +124,5 @@
   <!-- spinal -->
   <xacro:extra_module name = "fc" parent = "main_body" visible = "0" >
-    <origin xyz="${-rotor_x_middle} 0 0" rpy="0 0 0"/>
+    <origin xyz="${rotor_x_middle} 0 0" rpy="0 0 0"/>
     <inertial>
       <mass value = "0.05" />

Commit message: Add aero mobility 5DoF controller (temp)

File: robots/aero_mobility/urdf/robot.urdf.xacro (robot description, xacro)
@@ -6,4 +6,6 @@
   <thrust_link name="thrust" />
   <!-- kinematics [m] -->
+  <xacro:property name="PI" value="${3.14}" />
+  <xacro:property name="rotor_p_tilt" value="${20.0/180.0*PI}" />
   <xacro:property name="rotor_x_front" value="${1.2005}" />
   <xacro:property name="rotor_x_middle" value="${0.4005}" />
@@ -38,10 +40,10 @@
     </link>
   </xacro:macro>
-  <xacro:macro name="propeller_module" params="id x y z direction">
+  <xacro:macro name="propeller_module" params="id x y z roll pitch yaw direction">
     <joint name="rotor${id}" type="continuous">
       <limit effort="100.0" lower="${min_force}" upper="${max_force}" velocity="0.5"/>
       <parent link="main_body"/>
       <child link="thrust${id}"/>
-      <origin rpy="0 0 0" xyz="${x} ${y} ${z}"/>
+      <origin rpy="${roll} ${pitch} ${yaw}" xyz="${x} ${y} ${z}"/>
       <axis xyz="0 0 ${direction}"/>
     </joint>
@@ -57,5 +59,5 @@
       </inertial>
       <visual>
-        <origin rpy="0 0 0" xyz="0 0 0"/>
+        <origin rpy="${roll} ${pitch} ${yaw}" xyz="0 0 0"/>
         <geometry>
           <xacro:if value="${direction == 1}">
@@ -135,11 +137,11 @@
   </xacro:extra_module>
   <!-- propellers -->
-  <xacro:propeller_module id = "1" x = "${rotor_x_front}" y = "${rotor_y}" z = "${rotor_z}" direction = "1" />
-  <xacro:propeller_module id = "2" x = "${rotor_x_middle}" y = "${rotor_y}" z = "${rotor_z}" direction = "-1" />
-  <xacro:propeller_module id = "3" x = "${-rotor_x_middle}" y = "${rotor_y}" z = "${rotor_z}" direction = "1" />
-  <xacro:propeller_module id = "4" x = "${-rotor_x_front}" y = "${rotor_y}" z = "${rotor_z}"  direction = "-1" />
-  <xacro:propeller_module id = "5" x = "${-rotor_x_front}" y = "${-rotor_y}" z = "${rotor_z}" direction = "1" />
-  <xacro:propeller_module id = "6" x = "${-rotor_x_middle}" y = "${-rotor_y}" z = "${rotor_z}" direction = "-1" />
-  <xacro:propeller_module id = "7" x = "${rotor_x_middle}" y = "${-rotor_y}" z = "${rotor_z}" direction = "1" />
-  <xacro:propeller_module id = "8" x = "${rotor_x_front}" y = "${-rotor_y}" z = "${rotor_z}" direction = "-1" />
+  <xacro:propeller_module id = "1" x = "${rotor_x_front}" y = "${rotor_y}" z = "${rotor_z}" roll="0" pitch="${rotor_p_tilt}" yaw="0" direction = "1" />
+  <xacro:propeller_module id = "2" x = "${rotor_x_middle}" y = "${rotor_y}" z = "${rotor_z}" roll="0" pitch="${-rotor_p_tilt}" yaw="0" direction = "-1" />
+  <xacro:propeller_module id = "3" x = "${-rotor_x_middle}" y = "${rotor_y}" z = "${rotor_z}" roll="0" pitch="${rotor_p_tilt}" yaw="0" direction = "1" />
+  <xacro:propeller_module id = "4" x = "${-rotor_x_front}" y = "${rotor_y}" z = "${rotor_z}"  roll="0" pitch="${-rotor_p_tilt}" yaw="0" direction = "-1" />
+  <xacro:propeller_module id = "5" x = "${-rotor_x_front}" y = "${-rotor_y}" z = "${rotor_z}" roll="0" pitch="${-rotor_p_tilt}" yaw="0" direction = "1" />
+  <xacro:propeller_module id = "6" x = "${-rotor_x_middle}" y = "${-rotor_y}" z = "${rotor_z}" roll="0" pitch="${rotor_p_tilt}" yaw="0" direction = "-1" />
+  <xacro:propeller_module id = "7" x = "${rotor_x_middle}" y = "${-rotor_y}" z = "${rotor_z}" roll="0" pitch="${-rotor_p_tilt}" yaw="0" direction = "1" />
+  <xacro:propeller_module id = "8" x = "${rotor_x_front}" y = "${-rotor_y}" z = "${rotor_z}" roll="0" pitch="${rotor_p_tilt}" yaw="0" direction = "-1" />
 </robot>

Commit message: [Aero mobility] change rotor tilt angle arrangement

File: robots/aero_mobility/urdf/robot.urdf.xacro (robot description, xacro)
@@ -7,5 +7,5 @@
   <!-- kinematics [m] -->
   <xacro:property name="PI" value="${3.14}" />
-  <xacro:property name="rotor_p_tilt" value="${20.0/180.0*PI}" />
+  <xacro:property name="rotor_p_tilt" value="${-20.0/180.0*PI}" />
   <xacro:property name="rotor_x_front" value="${1.2005}" />
   <xacro:property name="rotor_x_middle" value="${0.4005}" />

Commit message: [Magic Carpet][Model] update the rotor tilt angle to improve the yaw controllability

File: robots/aero_mobility/urdf/robot.urdf.xacro (robot description, xacro)
@@ -7,5 +7,5 @@
   <!-- kinematics [m] -->
   <xacro:property name="PI" value="${3.14}" />
-  <xacro:property name="rotor_p_tilt" value="${-20.0/180.0*PI}" />
+  <xacro:property name="rotor_p_tilt" value="${20.0/180.0*PI}" />
   <xacro:property name="rotor_x_front" value="${1.2005}" />
   <xacro:property name="rotor_x_middle" value="${0.4005}" />

Commit message: [Magic Carpet] update urdf model to have livox mid360

File: robots/aero_mobility/urdf/robot.urdf.xacro (robot description, xacro)
@@ -136,4 +136,25 @@
     </inertial>
   </xacro:extra_module>
+  <!-- livox mid360 -->
+  <xacro:extra_module name = "lidar_imu" parent = "main_body" visible = "0" >
+    <origin xyz="${rotor_x_middle + 0.011} ${0.14 + 0.02329} ${0.015 + 0.047 - 0.04412}" rpy="0 0 0"/>
+    <inertial>
+      <mass value = "00" />
+      <origin xyz="0 0 0" rpy="0 0 0"/>
+      <inertia
+          ixx="0.0" ixy="0.0" ixz="0.0"
+          iyy="0.0" iyz="0.0" izz="0.0"/>
+    </inertial>
+  </xacro:extra_module>
+  <xacro:extra_module name = "livox_link" parent = "main_body" visible = "0" >
+    <origin xyz="${rotor_x_middle} 0.14 ${0.015 + 0.047}" rpy="0 0 0"/>
+    <inertial>
+      <mass value = "0" />
+      <origin xyz="0 0 0" rpy="0 0 0"/>
+      <inertia
+          ixx="0.0" ixy="0.0" ixz="0.0"
+          iyy="0.0" iyz="0.0" izz="0.0"/>
+    </inertial>
+  </xacro:extra_module>
   <!-- propellers -->
   <xacro:propeller_module id = "1" x = "${rotor_x_front}" y = "${rotor_y}" z = "${rotor_z}" roll="0" pitch="${rotor_p_tilt}" yaw="0" direction = "1" />

Commit message: [Magic Carpet] change rotor tilt and rotational directions

File: robots/aero_mobility/urdf/robot.urdf.xacro (robot description, xacro)
@@ -7,5 +7,5 @@
   <!-- kinematics [m] -->
   <xacro:property name="PI" value="${3.14}" />
-  <xacro:property name="rotor_p_tilt" value="${20.0/180.0*PI}" />
+  <xacro:property name="rotor_p_tilt" value="${-20.0/180.0*PI}" />
   <xacro:property name="rotor_x_front" value="${1.2005}" />
   <xacro:property name="rotor_x_middle" value="${0.4005}" />
@@ -158,11 +158,11 @@
   </xacro:extra_module>
   <!-- propellers -->
-  <xacro:propeller_module id = "1" x = "${rotor_x_front}" y = "${rotor_y}" z = "${rotor_z}" roll="0" pitch="${rotor_p_tilt}" yaw="0" direction = "1" />
-  <xacro:propeller_module id = "2" x = "${rotor_x_middle}" y = "${rotor_y}" z = "${rotor_z}" roll="0" pitch="${-rotor_p_tilt}" yaw="0" direction = "-1" />
-  <xacro:propeller_module id = "3" x = "${-rotor_x_middle}" y = "${rotor_y}" z = "${rotor_z}" roll="0" pitch="${rotor_p_tilt}" yaw="0" direction = "1" />
-  <xacro:propeller_module id = "4" x = "${-rotor_x_front}" y = "${rotor_y}" z = "${rotor_z}"  roll="0" pitch="${-rotor_p_tilt}" yaw="0" direction = "-1" />
-  <xacro:propeller_module id = "5" x = "${-rotor_x_front}" y = "${-rotor_y}" z = "${rotor_z}" roll="0" pitch="${-rotor_p_tilt}" yaw="0" direction = "1" />
-  <xacro:propeller_module id = "6" x = "${-rotor_x_middle}" y = "${-rotor_y}" z = "${rotor_z}" roll="0" pitch="${rotor_p_tilt}" yaw="0" direction = "-1" />
-  <xacro:propeller_module id = "7" x = "${rotor_x_middle}" y = "${-rotor_y}" z = "${rotor_z}" roll="0" pitch="${-rotor_p_tilt}" yaw="0" direction = "1" />
-  <xacro:propeller_module id = "8" x = "${rotor_x_front}" y = "${-rotor_y}" z = "${rotor_z}" roll="0" pitch="${rotor_p_tilt}" yaw="0" direction = "-1" />
+  <xacro:propeller_module id = "1" x = "${rotor_x_front}" y = "${rotor_y}" z = "${rotor_z}" roll="0" pitch="${rotor_p_tilt}" yaw="0" direction = "-1" />
+  <xacro:propeller_module id = "2" x = "${rotor_x_middle}" y = "${rotor_y}" z = "${rotor_z}" roll="0" pitch="${-rotor_p_tilt}" yaw="0" direction = "1" />
+  <xacro:propeller_module id = "3" x = "${-rotor_x_middle}" y = "${rotor_y}" z = "${rotor_z}" roll="0" pitch="${rotor_p_tilt}" yaw="0" direction = "-1" />
+  <xacro:propeller_module id = "4" x = "${-rotor_x_front}" y = "${rotor_y}" z = "${rotor_z}"  roll="0" pitch="${-rotor_p_tilt}" yaw="0" direction = "1" />
+  <xacro:propeller_module id = "5" x = "${-rotor_x_front}" y = "${-rotor_y}" z = "${rotor_z}" roll="0" pitch="${-rotor_p_tilt}" yaw="0" direction = "-1" />
+  <xacro:propeller_module id = "6" x = "${-rotor_x_middle}" y = "${-rotor_y}" z = "${rotor_z}" roll="0" pitch="${rotor_p_tilt}" yaw="0" direction = "1" />
+  <xacro:propeller_module id = "7" x = "${rotor_x_middle}" y = "${-rotor_y}" z = "${rotor_z}" roll="0" pitch="${-rotor_p_tilt}" yaw="0" direction = "-1" />
+  <xacro:propeller_module id = "8" x = "${rotor_x_front}" y = "${-rotor_y}" z = "${rotor_z}" roll="0" pitch="${rotor_p_tilt}" yaw="0" direction = "1" />
 </robot>

Commit message: [Magic Carpet][WIP] update weight model about battery

File: robots/aero_mobility/urdf/robot.urdf.xacro (robot description, xacro)
@@ -104,5 +104,6 @@
   <link name="main_body">
     <inertial>
-      <mass value = "${24.05 - 2.6 * 4}" />
+      <mass value = "${24.05}" />
+      <!-- <mass value = "${24.05 - 2.6 * 4}" /> -->
       <origin xyz="0 0 0" rpy="0 0 0"/>
       <inertia

Commit message: [Magic Carpet] update the robot URDF model with battery

File: robots/aero_mobility/urdf/robot.urdf.xacro (robot description, xacro)
@@ -158,4 +158,49 @@
     </inertial>
   </xacro:extra_module>
+  <!-- batteries -->
+  <xacro:extra_module name = "battery1" parent = "main_body" visible = "0" >
+    <origin xyz="0.18 0.5 0" rpy="0 0 0"/>
+    <inertial>
+      <mass value = "2.6" />
+      <origin xyz="0 0 0" rpy="0 0 0"/>
+      <inertia
+          ixx="0.01" ixy="0.0" ixz="0.0"
+          iyy="0.01" iyz="0.0"
+          izz="0.02"/>
+    </inertial>
+  </xacro:extra_module>
+  <xacro:extra_module name = "battery2" parent = "main_body" visible = "0" >
+    <origin xyz="-0.18 0.5 0" rpy="0 0 0"/>
+    <inertial>
+      <mass value = "2.6" />
+      <origin xyz="0 0 0" rpy="0 0 0"/>
+      <inertia
+          ixx="0.01" ixy="0.0" ixz="0.0"
+          iyy="0.01" iyz="0.0"
+          izz="0.02"/>
+    </inertial>
+  </xacro:extra_module>
+  <xacro:extra_module name = "battery3" parent = "main_body" visible = "0" >
+    <origin xyz="-0.18 -0.5 0" rpy="0 0 0"/>
+    <inertial>
+      <mass value = "2.6" />
+      <origin xyz="0 0 0" rpy="0 0 0"/>
+      <inertia
+          ixx="0.01" ixy="0.0" ixz="0.0"
+          iyy="0.01" iyz="0.0"
+          izz="0.02"/>
+    </inertial>
+  </xacro:extra_module>
+  <xacro:extra_module name = "battery4" parent = "main_body" visible = "0" >
+    <origin xyz="0.18 -0.5 0" rpy="0 0 0"/>
+    <inertial>
+      <mass value = "2.6" />
+      <origin xyz="0 0 0" rpy="0 0 0"/>
+      <inertia
+          ixx="0.01" ixy="0.0" ixz="0.0"
+          iyy="0.01" iyz="0.0"
+          izz="0.02"/>
+    </inertial>
+  </xacro:extra_module>
   <!-- propellers -->
   <xacro:propeller_module id = "1" x = "${rotor_x_front}" y = "${rotor_y}" z = "${rotor_z}" roll="0" pitch="${rotor_p_tilt}" yaw="0" direction = "-1" />

Commit message: [Kashiwa ESC][WIP] - remove battery model - disable livox and fast_lio / the ethernet config is also changed - takeoff height: 0.5m - [most important] modify the flight control gains: decrease position d gain; increase att LQI p gain

File: robots/aero_mobility/urdf/robot.urdf.xacro (robot description, xacro)
@@ -159,48 +159,48 @@
   </xacro:extra_module>
   <!-- batteries -->
-  <xacro:extra_module name = "battery1" parent = "main_body" visible = "0" >
-    <origin xyz="0.18 0.5 0" rpy="0 0 0"/>
-    <inertial>
-      <mass value = "2.6" />
-      <origin xyz="0 0 0" rpy="0 0 0"/>
-      <inertia
-          ixx="0.01" ixy="0.0" ixz="0.0"
-          iyy="0.01" iyz="0.0"
-          izz="0.02"/>
-    </inertial>
-  </xacro:extra_module>
-  <xacro:extra_module name = "battery2" parent = "main_body" visible = "0" >
-    <origin xyz="-0.18 0.5 0" rpy="0 0 0"/>
-    <inertial>
-      <mass value = "2.6" />
-      <origin xyz="0 0 0" rpy="0 0 0"/>
-      <inertia
-          ixx="0.01" ixy="0.0" ixz="0.0"
-          iyy="0.01" iyz="0.0"
-          izz="0.02"/>
-    </inertial>
-  </xacro:extra_module>
-  <xacro:extra_module name = "battery3" parent = "main_body" visible = "0" >
-    <origin xyz="-0.18 -0.5 0" rpy="0 0 0"/>
-    <inertial>
-      <mass value = "2.6" />
-      <origin xyz="0 0 0" rpy="0 0 0"/>
-      <inertia
-          ixx="0.01" ixy="0.0" ixz="0.0"
-          iyy="0.01" iyz="0.0"
-          izz="0.02"/>
-    </inertial>
-  </xacro:extra_module>
-  <xacro:extra_module name = "battery4" parent = "main_body" visible = "0" >
-    <origin xyz="0.18 -0.5 0" rpy="0 0 0"/>
-    <inertial>
-      <mass value = "2.6" />
-      <origin xyz="0 0 0" rpy="0 0 0"/>
-      <inertia
-          ixx="0.01" ixy="0.0" ixz="0.0"
-          iyy="0.01" iyz="0.0"
-          izz="0.02"/>
-    </inertial>
-  </xacro:extra_module>
+  <!-- <xacro:extra_module name = "battery1" parent = "main_body" visible = "0" > -->
+  <!--   <origin xyz="0.18 0.5 0" rpy="0 0 0"/> -->
+  <!--   <inertial> -->
+  <!--     <mass value = "2.6" /> -->
+  <!--     <origin xyz="0 0 0" rpy="0 0 0"/> -->
+  <!--     <inertia -->
+  <!--         ixx="0.01" ixy="0.0" ixz="0.0" -->
+  <!--         iyy="0.01" iyz="0.0" -->
+  <!--         izz="0.02"/> -->
+  <!--   </inertial> -->
+  <!-- </xacro:extra_module> -->
+  <!-- <xacro:extra_module name = "battery2" parent = "main_body" visible = "0" > -->
+  <!--   <origin xyz="-0.18 0.5 0" rpy="0 0 0"/> -->
+  <!--   <inertial> -->
+  <!--     <mass value = "2.6" /> -->
+  <!--     <origin xyz="0 0 0" rpy="0 0 0"/> -->
+  <!--     <inertia -->
+  <!--         ixx="0.01" ixy="0.0" ixz="0.0" -->
+  <!--         iyy="0.01" iyz="0.0" -->
+  <!--         izz="0.02"/> -->
+  <!--   </inertial> -->
+  <!-- </xacro:extra_module> -->
+  <!-- <xacro:extra_module name = "battery3" parent = "main_body" visible = "0" > -->
+  <!--   <origin xyz="-0.18 -0.5 0" rpy="0 0 0"/> -->
+  <!--   <inertial> -->
+  <!--     <mass value = "2.6" /> -->
+  <!--     <origin xyz="0 0 0" rpy="0 0 0"/> -->
+  <!--     <inertia -->
+  <!--         ixx="0.01" ixy="0.0" ixz="0.0" -->
+  <!--         iyy="0.01" iyz="0.0" -->
+  <!--         izz="0.02"/> -->
+  <!--   </inertial> -->
+  <!-- </xacro:extra_module> -->
+  <!-- <xacro:extra_module name = "battery4" parent = "main_body" visible = "0" > -->
+  <!--   <origin xyz="0.18 -0.5 0" rpy="0 0 0"/> -->
+  <!--   <inertial> -->
+  <!--     <mass value = "2.6" /> -->
+  <!--     <origin xyz="0 0 0" rpy="0 0 0"/> -->
+  <!--     <inertia -->
+  <!--         ixx="0.01" ixy="0.0" ixz="0.0" -->
+  <!--         iyy="0.01" iyz="0.0" -->
+  <!--         izz="0.02"/> -->
+  <!--   </inertial> -->
+  <!-- </xacro:extra_module> -->
   <!-- propellers -->
   <xacro:propeller_module id = "1" x = "${rotor_x_front}" y = "${rotor_y}" z = "${rotor_z}" roll="0" pitch="${rotor_p_tilt}" yaw="0" direction = "-1" />
