Commit message: [Dragon][Model][WIP] re-locate the fc frame on the root

File: robots/dragon/robots/quad/euclid_201709.urdf.xacro (robot description, xacro)
@@ -5,6 +5,6 @@
   <xacro:include filename="$(find dragon)/urdf/dragon_common.xacro" />
   <xacro:include filename="$(find dragon)/urdf/dragon_link.urdf.xacro" />
-  <xacro:dragon_module self="1" child="2" baselink="false" />
-  <xacro:dragon_module self="2" child="3" baselink="true" />
+  <xacro:dragon_module self="1" child="2" baselink="true" />
+  <xacro:dragon_module self="2" child="3" baselink="false" />
   <xacro:dragon_module self="3" child="4" baselink="false" />
   <xacro:dragon_module self="4" child="4" baselink="false" />

File: robots/dragon/urdf/dragon_link.urdf.xacro (robot description, xacro)
@@ -273,5 +273,5 @@
         <child link="fc"/>
         <parent link="link${self}"/>
-        <origin rpy="0 0 0" xyz="0.316 -0.004 0.043"/>
+        <origin rpy="0 0 0" xyz="0 0 0"/>
         <axis xyz="0 0 1"/>
       </joint>
