Commit message: Update

File: robots/hydrus_xi/urdf/common.xacro (robot description, xacro)
@@ -14,6 +14,6 @@
   <xacro:property name="rotor_radius" value=".0178"/>
   <!-- mass [Kg] -->
-  <xacro:property name="rotor_mass" value="0.02"/> <!-- exclude from center mass -->
-  <xacro:property name="bat_mass" value="0.193"/> <!-- 1300mAh -->
+  <xacro:property name="rotor_mass" value="0.15"/> <!-- exclude from center mass -->
+  <xacro:property name="bat_mass" value="0.0"/> <!-- 1300mAh -->
   <!-- dynamics -->
   <m_f_rate value="-0.0182" /> <!-- MN4010KV475_Afro_15inch -->
@@ -43,5 +43,5 @@
       <parent link="link4"/>
       <child link="end_effector"/>
-      <origin rpy="0 0 0" xyz="${link_length} 0 0"/>
+      <origin rpy="0 0 0" xyz="${link_length} 0 0.04"/>
   </joint>
   <!-- <link name="end_effector">
@@ -82,10 +82,4 @@
         </geometry>
       </collision>
-      <collision>
-        <origin rpy="0 0 0" xyz="0.2 0 0"/>
-        <geometry>
-          <sphere radius="0.01"/>
-        </geometry>
-      </collision>
       <visual>
         <origin rpy="0 1.57 0" xyz="0.1 0 0"/>
@@ -114,8 +108,8 @@
       </collision>
   </link>
-  <gazebo reference="end_effector">
+  <gazebo reference="end_frame">
     <sensor name="contacts" type="contact">
         <contact>
-          <collision>link4_fixed_joint_lump__end_effector_collision_2</collision>
+          <collision>link4_fixed_joint_lump__end_frame_collision_2</collision>
         </contact>
         <plugin name="gazebo_ros_bumper_controller" filename="libgazebo_ros_bumper.so">

File: robots/hydrus_xi/urdf/curved_wall.urdf (robot description, URDF)
Before this commit: robot curved_wall, 1 links, 0 joints
Links:
- link curved_wall: geometry collision cylinder length=4 radius=1.2; visual cylinder length=4 radius=1.2

File: robots/hydrus_xi/urdf/link.urdf.xacro (robot description, xacro)
@@ -8,5 +8,5 @@
         <inertial>
           <origin xyz="0.286949 -0.000071 0.011024" rpy="0 0 0"/>
-          <mass value="0.535052"/>
+          <mass value="0.575052"/>
           <inertia
               ixx="0.000808" iyy="0.012747" izz="0.012027"
@@ -21,5 +21,5 @@
         <inertial>
           <origin xyz="0.327173 -0.000033 -0.006011" rpy="0 0 0"/>
-          <mass value="0.455151"/>
+          <mass value="0.495151"/>
           <inertia
               ixx="0.001020" iyy="0.008076" izz="0.007129"
@@ -34,5 +34,5 @@
         <inertial>
           <origin xyz="0.256002 -0.000077 0.010307" rpy="0 0 0"/>
-          <mass value="0.491782"/>
+          <mass value="0.531782"/>
           <inertia
               ixx="0.000785" iyy="0.007046" izz="0.006334"
@@ -51,5 +51,5 @@
       <inertial>
         <origin xyz="-0.006114 0.000001 0.032778" rpy="0 0 0"/>
-        <mass value="0.260"/>
+        <mass value="0.130"/>
         <inertia
             ixx="0.001" iyy="0.001" izz="0.001"

Commit message: Add comments for admittance control

File: robots/hydrus_xi/urdf/common.xacro (robot description, xacro)
@@ -14,11 +14,6 @@
   <xacro:property name="rotor_radius" value=".0178"/>
   <!-- mass [Kg] -->
-<<<<<<< HEAD
-  <xacro:property name="rotor_mass" value="0.15"/> <!-- exclude from center mass -->
-  <xacro:property name="bat_mass" value="0.0"/> <!-- 1300mAh -->
-=======
   <xacro:property name="rotor_mass" value="0.02"/> <!-- exclude from center mass -->
   <xacro:property name="bat_mass" value="0.05"/> <!-- 1300mAh -->
->>>>>>> 9dc48a1715533e59d0ea7771f1561de774bd206d
   <!-- dynamics -->
   <m_f_rate value="-0.0182" /> <!-- MN4010KV475_Afro_15inch -->
