Commit message: Add admittance control(IK part)

File: robots/dragon/urdf/v1_5/dragon_common.xacro (robot description, xacro)
@@ -51,4 +51,10 @@
     </link>
   </xacro:macro>
+  <link name="end_frame"/>
+  <joint name="end_eff" type="fixed">
+      <parent link="link4"/>
+      <child link="end_frame"/>
+      <origin rpy="0 0 0" xyz="${link_length} 0 0"/>
+  </joint>
   <!-- friction -->
   <xacro:macro name="friction" params="self">

Commit message: commit

File: robots/dragon/urdf/v1_5/dragon_common.xacro (robot description, xacro)
@@ -33,4 +33,19 @@
     </visual>
   </xacro:macro>
+  <gazebo reference="link4">
+    <sensor name="contacts" type="contact">
+        <contact>
+          <collision>link4_fixed_joint_lump__end_frame_collision_1</collision>
+        </contact>
+        <plugin name="gazebo_ros_bumper_controller" filename="libgazebo_ros_bumper.so">
+          <always_on>true</always_on>
+          <robotNamespace>/dragon</robotNamespace>
+          <bumperTopicName>bumper_states</bumperTopicName>
+          <frameName>bumper</frameName>
+          <visualize>true</visualize>
+          <update_rate>1000.0</update_rate>
+        </plugin>
+    </sensor>
+  </gazebo>
   <xacro:macro name="extra_module" params="name parent *origin *inertial visible:=0 model_url:=1 scale:=1">
     <joint name="${parent}2${name}" type="fixed">
@@ -51,5 +66,12 @@
     </link>
   </xacro:macro>
-  <link name="end_frame"/>
+  <link name="end_frame">
+   <collision>
+        <origin rpy="0 0 0" xyz="0 0 0"/>
+        <geometry>
+          <sphere radius="0.1"/>
+        </geometry>
+      </collision>
+  </link>
   <joint name="end_eff" type="fixed">
       <parent link="link4"/>

Commit message: visulize end effector

File: robots/dragon/urdf/v1_5/dragon_common.xacro (robot description, xacro)
@@ -70,7 +70,13 @@
         <origin rpy="0 0 0" xyz="0 0 0"/>
         <geometry>
-          <sphere radius="0.1"/>
+          <sphere radius="0.02"/>
         </geometry>
       </collision>
+      <visual>
+      <origin rpy="0 0 0" xyz="0 0 0"/>
+        <geometry>
+          <sphere radius="0.02"/>
+        </geometry>
+    </visual>
   </link>
   <joint name="end_eff" type="fixed">
