Commit message: Ready for exp

File: robots/dragon/urdf/v1_5/dragon_common.xacro (robot description, xacro)
@@ -85,4 +85,31 @@
       <origin rpy="0 0 0" xyz="${link_length} 0 0"/>
   </joint>
+  <link name="end">
+   <inertial>
+          <origin xyz="0 0 0" rpy="0 0 0"/>
+          <mass value="0.001" />
+          <inertia
+              ixx="0.0001" iyy="0.0001" izz="0.0001"
+              ixy="0.0000" ixz="0.0000" iyz="0.0000"/>
+        </inertial>
+   <collision>
+        <origin rpy="0 0 0" xyz="0 0 0"/>
+        <geometry>
+          <sphere radius="0.02"/>
+        </geometry>
+      </collision>
+      <visual>
+      <origin rpy="0 0 0" xyz="0 0 0"/>
+        <geometry>
+          <sphere radius="0.02"/>
+        </geometry>
+    </visual>
+  </link>
+  <joint name="end_joint" type="continuous">
+      <parent link="link4"/>
+      <child link="end"/>
+      <origin rpy="0 0 0" xyz="${link_length} 0 0"/>
+      <axis xyz="0 0 1"/>
+  </joint>
   <!-- friction -->
   <xacro:macro name="friction" params="self">

Commit message: Successfully experiments in basic movement and single joint deformation

File: robots/dragon/urdf/v1_5/dragon_common.xacro (robot description, xacro)
@@ -88,5 +88,5 @@
    <inertial>
           <origin xyz="0 0 0" rpy="0 0 0"/>
-          <mass value="0.001" />
+          <mass value="0.05" />
           <inertia
               ixx="0.0001" iyy="0.0001" izz="0.0001"
